Commit message: Reducing agv mesh and fixing urdf definition

File: robot/agvota/urdf/agv_base.urdf.xacro (robot description, xacro)
@@ -7,5 +7,5 @@
         <origin xyz="0 0 -0.1625" rpy=" 0 0 0"/>
         <geometry>
-          <mesh filename="package://arena-simulation-setup/robot/agv-ota/meshes/OTAv07_meshes/OTA-v0.7.stl" scale="0.001 0.001 0.001"/>
+          <mesh filename="package://arena-simulation-setup/robot/agvota/meshes/OTAv07_meshes/OTA-v0.7.stl" scale="0.001 0.001 0.001"/>
         </geometry>
       </visual>
@@ -13,5 +13,5 @@
         <origin xyz="0 0 -0.075" rpy=" 0 0 0"/>
         <geometry>
-          <!--<mesh filename="package://arena-simulation-setup/robot/agv-ota/meshes/OTAv07_meshes/OTA-v0.7.stl" scale="0.001 0.001 0.001"/> -->
+          <!--<mesh filename="package://arena-simulation-setup/robot/agvota/meshes/OTAv07_meshes/OTA-v0.7.stl" scale="0.001 0.001 0.001"/> -->
           <box size="1.02 0.72 0.14"/>
         </geometry>
@@ -27,5 +27,5 @@
         <origin xyz="0 0 0" rpy="1.570796 0 -1.570796"/>
         <geometry>
-          <mesh filename="package://arena-simulation-setup/robot/agv-ota/meshes/OTAv07_meshes/S30B-XXXXXX.stl" scale="0.001 0.001 0.001"/>
+          <mesh filename="package://arena-simulation-setup/robot/agvota/meshes/OTAv07_meshes/S30B-XXXXXX.stl" scale="0.001 0.001 0.001"/>
         </geometry>
       </visual>
@@ -33,5 +33,5 @@
         <origin xyz="0 0 0.0" rpy="1.570796 0 -1.570796"/>
         <geometry>
-          <mesh filename="package://arena-simulation-setup/robot/agv-ota/meshes/OTAv07_meshes/S30B-XXXXXX.stl" scale="0.001 0.001 0.001"/>
+          <mesh filename="package://arena-simulation-setup/robot/agvota/meshes/OTAv07_meshes/S30B-XXXXXX.stl" scale="0.001 0.001 0.001"/>
         </geometry>
       </collision>  -->
@@ -82,5 +82,5 @@
           <origin xyz="0 0 0" rpy="0 0 0"/>
           <geometry>
-            <mesh filename="package://arena-simulation-setup/robot/agv-ota/meshes/OTAv07_meshes/zed.stl" />
+            <mesh filename="package://arena-simulation-setup/robot/agvota/meshes/OTAv07_meshes/zed.stl" />
           </geometry>
           <material name="black">
@@ -91,5 +91,5 @@
           <origin xyz="0 0 0" rpy="0 0 0"/>
           <geometry>
-            <mesh filename="package://arena-simulation-setup/robot/agv-ota/meshes/OTAv07_meshes/ZED.stl" />
+            <mesh filename="package://arena-simulation-setup/robot/agvota/meshes/OTAv07_meshes/ZED.stl" />
           </geometry>
           <material name="light_grey">

File: robot/agvota/urdf/agv_caster.urdf.xacro (robot description, xacro)
@@ -7,5 +7,5 @@
         <origin xyz="0 0 0" rpy=" 0 0 0"/>
         <geometry>
-          <mesh filename="package://arena-simulation-setup/robot/agv-ota/meshes/OTAv07_meshes/SarhosTeker.stl" scale="0.001 0.001 0.001"/>
+          <mesh filename="package://arena-simulation-setup/robot/agvota/meshes/OTAv07_meshes/SarhosTeker.stl" scale="0.001 0.001 0.001"/>
         </geometry>
       </visual>

File: robot/agvota/urdf/agv_ir.urdf.xacro (robot description, xacro)
@@ -11,5 +11,5 @@
 			<origin xyz="0 0 0" rpy="0 0 0"/>
 			<geometry>
-				<mesh filename="package://arena-simulation-setup/robot/agv-ota/meshes/OTAv07_meshes/FotoelektrikSensor.stl" scale="0.0015 0.0015 0.0015"/>
+				<mesh filename="package://arena-simulation-setup/robot/agvota/meshes/OTAv07_meshes/FotoelektrikSensor.stl" scale="0.0015 0.0015 0.0015"/>
 			</geometry>
 		</visual>

File: robot/agvota/urdf/agv_wheel.urdf.xacro (robot description, xacro)
@@ -6,5 +6,5 @@
         <origin xyz="0 0 0" rpy=" 0 0 1.570796"/>
         <geometry>
-          <mesh filename="package://arena-simulation-setup/robot/agv-ota/meshes/OTAv07_meshes/AnaTeker.stl" scale="0.001 0.001 0.001"/>
+          <mesh filename="package://arena-simulation-setup/robot/agvota/meshes/OTAv07_meshes/AnaTeker.stl" scale="0.001 0.001 0.001"/>
         </geometry>
       </visual>
