Commit message: merge from jacenty | updated gazebo robot models to be compatible with marl setup and publish to topics with namespaces
tiago, youbot and cob4 still todo

File: robot/agvota/urdf/agv_base.urdf.xacro (robot description, xacro)
@@ -72,6 +72,6 @@
         <plugin name="laser_scan_plugin" filename="libgazebo_ros_laser.so">
             <topicName>scan</topicName>
-            <frameName>scan_link</frameName>
-            <tf_prefix>/</tf_prefix>
+            <frameName>${robot_namespace}_base_footprint</frameName>
+            <!-- <tf_prefix>${robot_namespace}</tf_prefix> -->
         </plugin>
       </sensor>

File: robot/agvota/urdf/agv_plugin.urdf.xacro (robot description, xacro)
@@ -26,9 +26,9 @@
         <wheelTorque>20</wheelTorque>
         <wheelAcceleration>1.8</wheelAcceleration>
-        <commandTopic>cmd_vel</commandTopic>
-        <odometryTopic>odom</odometryTopic>
-        <odometryFrame>odom</odometryFrame>
+        <commandTopic>${robot_namespace}/cmd_vel</commandTopic>
+        <odometryTopic>${robot_namespace}/odom</odometryTopic>
+        <odometryFrame>${robot_namespace}_odom</odometryFrame>
         <odometrySource>world</odometrySource>
-        <robotBaseFrame>base_link</robotBaseFrame>
+        <robotBaseFrame>${robot_namespace}_base_footprint</robotBaseFrame>
 	      <legacyMode>true</legacyMode>
 	      <publishTf>true</publishTf>

File: robot/agvota/urdf/agvota.urdf.xacro (robot description, xacro)
@@ -1,4 +1,6 @@
 <?xml version="1.0"?>
 <robot name="agvota" xmlns:xacro="http://ros.org/wiki/xacro">
+	<xacro:arg name="robot_namespace" default="$(optenv ROBOT_NAMESPACE /)" />
+	<xacro:property name="robot_namespace" value="$(arg robot_namespace)" />
 	<xacro:include filename="$(find arena-simulation-setup)/robot/agvota/urdf/agv_base.urdf.xacro"/>
 	<xacro:include filename="$(find arena-simulation-setup)/robot/agvota/urdf/inertia_tensors.urdf.xacro"/>

File: robot/cob4/urdf/cob4.urdf.xacro (robot description, xacro)
@@ -2,4 +2,6 @@
 <robot xmlns:xacro="http://www.ros.org/wiki/xacro"
        name="cob4-11" >
+	<xacro:arg name="robot_namespace" default="$(optenv ROBOT_NAMESPACE /)" />
+	<xacro:property name="robot_namespace" value="$(arg robot_namespace)" />
   <!-- common stuff -->
   <xacro:include filename="$(find arena-simulation-setup)/robot/cob4/cob_description/urdf/common.xacro" />
@@ -12,13 +14,13 @@
   <xacro:include filename="$(find arena-simulation-setup)/robot/cob4/cob_description/urdf/sensors/sick_s300_laser.urdf.xacro"/>
   <!-- composition of the robot -->
-  <xacro:base name="base"/>
+  <xacro:base name="${robot_namespace}_base"/>
   <!-- laser scanners -->
-  <xacro:sick_s300_laser_v0 name="base_laser_front" parent="base">
+  <xacro:sick_s300_laser_v0 name="base_laser_front" parent="${robot_namespace}_base">
     <origin xyz="${laser_front_x} ${laser_front_y} ${laser_front_z}" rpy="${laser_front_roll} ${laser_front_pitch} ${laser_front_yaw}" />
   </xacro:sick_s300_laser_v0>
-  <xacro:sick_s300_laser_v0 name="base_laser_left" parent="base">
+  <xacro:sick_s300_laser_v0 name="base_laser_left" parent="${robot_namespace}_base">
     <origin xyz="${laser_left_x} ${laser_left_y} ${laser_left_z}" rpy="${laser_left_roll} ${laser_left_pitch} ${laser_left_yaw}" />
   </xacro:sick_s300_laser_v0>
-  <xacro:sick_s300_laser_v0 name="base_laser_right" parent="base">
+  <xacro:sick_s300_laser_v0 name="base_laser_right" parent="${robot_namespace}_base">
     <origin xyz="${laser_right_x} ${laser_right_y} ${laser_right_z}" rpy="${laser_right_roll} ${laser_right_pitch} ${laser_right_yaw}" />
   </xacro:sick_s300_laser_v0>

File: robot/dingo/urdf/accessories.urdf.xacro (robot description, xacro)
@@ -19,5 +19,5 @@
   -->
   <xacro:if value="$(optenv DINGO_LASER 1)">
-    <xacro:property name="lidar_model" value="$(optenv DINGO_LASER_MODEL lms1xx)" />
+    <xacro:property name="lidar_model" value="$(optenv DINGO_LASER_MODEL ust10)" />
     <!-- <xacro:if value="${lidar_model == 'lms1xx'}">
       <xacro:sick_lms1xx_mount prefix="$(optenv DINGO_LASER_MOUNT front)"

File: robot/dingo/urdf/accessories/hokuyo_ust10.urdf.xacro (robot description, xacro)
@@ -42,4 +42,5 @@
             <topicName>${topic}</topicName>
             <frameName>${frame}</frameName>
+            <tf_prefix>${robot_namespace}</tf_prefix>
             <robotNamespace>${robot_namespace}</robotNamespace>
           </plugin>
@@ -47,5 +48,5 @@
       </gazebo>
     </xacro:macro>
-    <xacro:hokuyo_ust10 frame="${prefix}_laser" topic="${topic}" />
+    <xacro:hokuyo_ust10 frame="${robot_namespace}_base_footprint" topic="${robot_namespace}/${topic}" robot_namespace="${robot_namespace}" />
     <link name="${prefix}_laser_mount">
       <visual>
@@ -62,5 +63,5 @@
       <origin xyz="0 0 0.055" rpy="0 0 0" />
       <parent link="${prefix}_laser_mount" />
-      <child link="${prefix}_laser" />
+      <child link="${robot_namespace}_base_footprint" />
     </joint>
     <gazebo reference="${prefix}_laser_mount">

File: robot/dingo/urdf/dingo.urdf.xacro (robot description, xacro)
@@ -1,4 +1,251 @@
 <?xml version="1.0"?>
 <robot name="dingo" xmlns:xacro="http://www.ros.org/wiki/xacro">
-  <xacro:include filename="$(find arena-simulation-setup)/robot/dingo/urdf/dingo-d.urdf.xacro" />
+	<xacro:arg name="robot_namespace" default="$(optenv ROBOT_NAMESPACE /)" />
+	<xacro:property name="robot_namespace" value="$(arg robot_namespace)" />
+	<xacro:property name="PI" value="3.1415926535897931" />
+	<xacro:property name="wheel_radius" value="0.049" />
+	<xacro:property name="wheel_mass" value="0.111" />
+	<xacro:property name="wheel_width" value="0.02032" />
+	<xacro:property name="wheel_x_offset" value="0.0989838" />
+	<xacro:property name="wheel_z_offset" value="0.0345" />
+	<xacro:property name="wheelbase" value="0.2160016" />
+	<xacro:property name="dummy_inertia" value="1e-09"/>
+	<material name="dark_grey"><color rgba="0.2 0.2 0.2 1.0" /></material>
+	<material name="light_grey"><color rgba="0.4 0.4 0.4 1.0" /></material>
+	<material name="yellow"><color rgba="0.8 0.8 0.0 1.0" /></material>
+	<material name="black"><color rgba="0.15 0.15 0.15 1.0" /></material>
+	<xacro:macro name="wheel" params="prefix *joint_pose">
+		<link name="${prefix}_wheel_link">
+		<visual>
+			<origin xyz="0 0 0" rpy="0 0 0"/>
+			<geometry>
+			<mesh filename="package://arena-simulation-setup/robot/dingo/meshes/wheel.stl"/>
+			</geometry>
+			<material name="black" />
+		</visual>
+		<collision>
+			<origin xyz="0 0 0" rpy="${PI/2} 0 0"/>
+			<geometry>
+			<cylinder radius="${wheel_radius}" length="${wheel_width}"/>
+			</geometry>
+		</collision>
+		<inertial>
+			<origin xyz="0 0 0" rpy="0 0 0"/>
+			<mass value="${wheel_mass}"/>
+			<inertia
+			ixx="0.0003234" ixy="0" ixz="0"
+			iyy="0.0003234" iyz="0"
+			izz="0.00049015"/>
+		</inertial>
+		</link>
+		<gazebo reference="${prefix}_wheel_link">
+		<material>Gazebo/DarkGrey</material>
+		<selfCollide>false</selfCollide>
+		<mu1 value="0.5"/>
+		<mu2 value="0.5"/>
+		<kp value="10000000.0" />
+		<kd value="1" />
+		<fdir1 value="1 0 0"/>
+		</gazebo>
+		<joint name="${prefix}_wheel" type="continuous">
+		<parent link="chassis_link"/>
+		<child link="${prefix}_wheel_link" />
+		<xacro:insert_block name="joint_pose" />
+		<axis xyz="0 1 0" />
+		</joint>
+		<transmission name="${prefix}_wheel_trans">
+		<type>transmission_interface/SimpleTransmission</type>
+		<joint name="${prefix}_wheel">
+			<hardwareInterface>hardware_interface/VelocityJointInterface</hardwareInterface>
+		</joint>
+		<actuator name="${prefix}_actuator">
+			<mechanicalReduction>1</mechanicalReduction>
+		</actuator>
+		</transmission>
+	</xacro:macro>
+	<xacro:wheel prefix="left">
+		<origin xyz="${wheel_x_offset} ${wheelbase+wheel_width/2} ${wheel_z_offset}" rpy="0 0 0" />
+	</xacro:wheel>
+	<xacro:wheel prefix="right">
+		<origin xyz="${wheel_x_offset} ${-wheelbase-wheel_width/2} ${wheel_z_offset}" rpy="0 0 0" />
+	</xacro:wheel>
+	<link name="rear_caster">
+		<visual>
+		<origin rpy="0 0 0" xyz="0 0 0"/>
+		<geometry>
+			<sphere radius="0.01"/>
+		</geometry>
+		<material name="black"/>
+		</visual>
+		<collision>
+		<geometry>
+			<sphere radius="0.01"/>
+		</geometry>
+		<origin rpy="0 0 0" xyz="0 0 0"/>
+		<surface>
+			<friction>
+			<ode>
+				<mu>0.0</mu>
+				<mu2>0.0</mu2>
+				<slip1>1.0</slip1>
+				<slip2>1.0</slip2>
+			</ode>
+			</friction>
+		</surface>
+		</collision>
+		<inertial>
+		<mass value="0.1" />
+		<origin xyz="0 0 0" />
+		<inertia ixx="0.001" ixy="0.0" ixz="0.0"
+				iyy="0.001" iyz="0.0"
+				izz="0.001" />
+		</inertial>
+	</link>
+	<joint name="rear_caster_joint" type="fixed">
+		<parent link="chassis_link"/>
+		<child link="rear_caster"/>
+		<origin xyz="-0.244 0 -0.00674" rpy="0 0 0"/>
+	</joint>
+	<gazebo reference="rear_caster">
+		<turnGravityOff>false</turnGravityOff>
+		<kp>1000000.0</kp>
+		<kd>100.0</kd>
+		<mu1>0.2</mu1>
+		<mu2>0.2</mu2>
+		<fdir1>1 0 0</fdir1>
+		<minDepth>0.00</minDepth>
+		<implicitSpringDamper>1</implicitSpringDamper>
+	</gazebo>
+	<link name="base_link"></link>
+	<joint name="base_link_joint" type="fixed">
+		<origin xyz="0 0 0" rpy="0 0 0" />
+		<parent link="base_link"/>
+		<child link="chassis_link" />
+	</joint>
+	<link name="chassis_link">
+		<visual>
+		<origin xyz="0 0 0" rpy="0 0 0"/>
+		<geometry>
+			<mesh filename="package://arena-simulation-setup/robot/dingo/meshes/diff_chassis.dae"/>
+		</geometry>
+		</visual>
+		<collision>
+		<origin xyz="0 0 0"/>
+		<geometry>
+			<mesh filename="package://arena-simulation-setup/robot/dingo/meshes/diff_chassis_collision.stl"/>
+		</geometry>
+		</collision>
+		<inertial>
+		<!-- Center of mass -->
+		<origin xyz="0 0 0" rpy="0 0 0"/>
+		<mass value="10.0"/>
+		<!-- Moments of inertia: ( chassis without wheels ) -->
+		<inertia
+			ixx="0.2216" ixy="0" ixz="0"
+			iyy="0.2458" iyz="0"
+			izz="0.4474"/>
+		</inertial>
+	</link>
+	<link name="imu_link">
+		<inertial>
+		<mass value="0.001"/>
+		<origin xyz="0 0 0" rpy="0 0 0"/>
+		<inertia ixx="${dummy_inertia}" ixy="0.0" ixz="0.0" iyy="${dummy_inertia}" iyz="0.0" izz="${dummy_inertia}"/>
+		</inertial>
+	</link>
+	<joint name="imu_joint" type="fixed">
+		<parent link="chassis_link" />
+		<child link="imu_link" />
+	</joint>
+	<!--
+		Mounting points for accessories in the top channel.
+		These are flush with the top of the robot and all oriented to face forwards.
+		Dingo-D has 6 evenly-spaced 80mm mounts
+		We name the mounts (from front to back)
+		- front
+		- front b
+		- front c
+		- rear c
+		- rear b
+		- rear
+	-->
+	<link name="front_mount"/>
+	<link name="front_b_mount"/>
+	<link name="front_c_mount"/>
+	<link name="rear_mount"/>
+	<link name="rear_b_mount"/>
+	<link name="rear_c_mount"/>
+	<joint name="front_c_mount_joint" type="fixed">
+		<origin xyz="0.040 0 0.064263" rpy="0 0 0" />
+		<parent link="chassis_link"/>
+		<child link="front_c_mount" />
+	</joint>
+	<joint name="front_b_mount_joint" type="fixed">
+		<origin xyz="0.080 0 0" rpy="0 0 0" />
+		<parent link="front_c_mount"/>
+		<child link="front_b_mount" />
+	</joint>
+	<joint name="front_mount_joint" type="fixed">
+		<origin xyz="0.080 0 0" rpy="0 0 0" />
+		<parent link="front_b_mount"/>
+		<child link="front_mount" />
+	</joint>
+	<joint name="rear_c_mount_joint" type="fixed">
+		<origin xyz="-0.040 0 0.064263" rpy="0 0 0" />
+		<parent link="chassis_link"/>
+		<child link="rear_c_mount" />
+	</joint>
+	<joint name="rear_b_mount_joint" type="fixed">
+		<origin xyz="-0.080 0 0" rpy="0 0 0" />
+		<parent link="rear_c_mount"/>
+		<child link="rear_b_mount" />
+	</joint>
+	<joint name="rear_moint_joint" type="fixed">
+		<origin xyz="-0.080 0 0" rpy="0 0 0" />
+		<parent link="rear_b_mount"/>
+		<child link="rear_mount" />
+	</joint>
+	<!--
+		Mounting point for accessories on the front bumper.
+		Use with caution, but thin sensors (e.g Raspberry Pi NoIR camera) could
+		be mounted here for low-budget, front-facing capabilities
+	-->
+	<link name="front_bumper_mount"></link>
+	<joint name="front_bumper_mount_joint" type="fixed">
+		<origin xyz="0.274 0 0.0345125" rpy="0 0 0" />
+		<parent link="chassis_link"/>
+		<child link="front_bumper_mount" />
+	</joint>
+	<gazebo>
+		<plugin name="gazebo_ros_control" filename="libgazebo_ros_control.so">
+		<robotNamespace>${robot_namespace}</robotNamespace>
+		</plugin>
+	</gazebo>
+	<gazebo>
+		<plugin name="imu_controller" filename="libhector_gazebo_ros_imu.so">
+		<robotNamespace>${robot_namespace}</robotNamespace>
+		<updateRate>50.0</updateRate>
+		<bodyName>imu_link</bodyName>
+		<topicName>imu/data</topicName>
+		<accelDrift>0.005 0.005 0.005</accelDrift>
+		<accelGaussianNoise>0.005 0.005 0.005</accelGaussianNoise>
+		<rateDrift>0.005 0.005 0.005 </rateDrift>
+		<rateGaussianNoise>0.005 0.005 0.005 </rateGaussianNoise>
+		<headingDrift>0.005</headingDrift>
+		<headingGaussianNoise>0.005</headingGaussianNoise>
+		</plugin>
+	</gazebo>
+	<gazebo reference="base_link">
+		<turnGravityOff>false</turnGravityOff>
+	</gazebo>
+	<gazebo reference="chassis_link">
+		<turnGravityOff>false</turnGravityOff>
+	</gazebo>
+	<gazebo reference="imu_link">
+		<turnGravityOff>false</turnGravityOff>
+	</gazebo>
+	<!-- Optional standard accessories, including their simulation data. The rendering
+		of these into the final description is controlled by optenv variables, which
+		default each one to off.-->
+	<xacro:include filename="$(find arena-simulation-setup)/robot/dingo/urdf/accessories.urdf.xacro" />
 </robot>

File: robot/jackal/urdf/accessories/hokuyo_ust10.urdf.xacro (robot description, xacro)
@@ -39,4 +39,5 @@
             <topicName>${topic}</topicName>
             <frameName>${frame}</frameName>
+            <tf_prefix>${robot_namespace}</tf_prefix>
             <robotNamespace>${robot_namespace}</robotNamespace>
           </plugin>
@@ -44,5 +45,5 @@
       </gazebo>
     </xacro:macro>
-    <xacro:hokuyo_ust10 frame="${prefix}_laser" topic="${topic}"/>
+    <xacro:hokuyo_ust10 frame="${robot_namespace}_base_footprint" topic="${robot_namespace}/${topic}" robot_namespace="${robot_namespace}" />
     <joint name="${prefix}_laser_mount_joint" type="fixed">
       <xacro:insert_block name="origin" />
@@ -64,5 +65,5 @@
       <origin xyz="0 0 0.0474" rpy="0 0 0" />
       <parent link="${prefix}_laser_mount" />
-      <child link="${prefix}_laser" />
+      <child link="${robot_namespace}_base_footprint" />
     </joint>
     <gazebo reference="${prefix}_laser_mount">

File: robot/jackal/urdf/jackal.urdf.xacro (robot description, xacro)
@@ -2,4 +2,5 @@
 <robot name="jackal" xmlns:xacro="http://www.ros.org/wiki/xacro">
   <xacro:property name="PI" value="3.1415926535897931" />
+  <xacro:arg name="robot_namespace" default="$(optenv ROBOT_NAMESPACE /)" />
   <xacro:property name="wheelbase" value="0.262" />
   <xacro:property name="track" value="0.37559" />
@@ -13,4 +14,5 @@
   <xacro:property name="dummy_inertia" value="1e-09"/>
   <xacro:property name="mount_spacing" value="0.120" />
+  <xacro:property name="robot_namespace" value="$(arg robot_namespace)" />
   <material name="dark_grey"><color rgba="0.2 0.2 0.2 1.0" /></material>
   <material name="light_grey"><color rgba="0.4 0.4 0.4 1.0" /></material>
@@ -80,8 +82,8 @@
     <origin xyz="${-wheelbase/2} ${-track/2} ${wheel_vertical_offset}" rpy="0 0 0" />
   </xacro:wheel>
-  <link name="base_link"></link>
-  <joint name="base_link_joint" type="fixed">
+  <link name="base_footprint"></link>
+  <joint name="base_footprint_joint" type="fixed">
     <origin xyz="0 0 0" rpy="0 0 0" />
-    <parent link="base_link"/>
+    <parent link="base_footprint"/>
     <child link="chassis_link" />
   </joint>
@@ -221,4 +223,38 @@
     <origin xyz="${mount_spacing} 0 0" />
   </joint>
+  <gazebo>
+    <plugin name="gazebo_ros_control" filename="libgazebo_ros_control.so">
+      <robotNamespace>${robot_namespace}</robotNamespace>
+    </plugin>
+  </gazebo>
+  <gazebo>
+    <plugin name="imu_controller" filename="libhector_gazebo_ros_imu.so">
+      <robotNamespace>${robot_namespace}</robotNamespace>
+      <updateRate>50.0</updateRate>
+      <bodyName>imu_link</bodyName>
+      <topicName>imu/data</topicName>
+      <accelDrift>0.005 0.005 0.005</accelDrift>
+      <accelGaussianNoise>0.005 0.005 0.005</accelGaussianNoise>
+      <rateDrift>0.005 0.005 0.005 </rateDrift>
+      <rateGaussianNoise>0.005 0.005 0.005 </rateGaussianNoise>
+      <headingDrift>0.005</headingDrift>
+      <headingGaussianNoise>0.005</headingGaussianNoise>
+    </plugin>
+  </gazebo>
+  <gazebo>
+    <plugin name="gps_controller" filename="libhector_gazebo_ros_gps.so">
+      <updateRate>40</updateRate>
+      <robotNamespace>${robot_namespace}</robotNamespace>
+      <bodyName>navsat_link</bodyName>
+      <frameId>${robot_namespace}_base_footprint</frameId>
+      <topicName>/navsat/fix</topicName>
+      <velocityTopicName>/navsat/vel</velocityTopicName>
+      <referenceLatitude>49.9</referenceLatitude>
+      <referenceLongitude>8.9</referenceLongitude>
+      <referenceHeading>0</referenceHeading>
+      <referenceAltitude>0</referenceAltitude>
+      <drift>0.0001 0.0001 0.0001</drift>
+    </plugin>
+  </gazebo>
   <!-- Bring in simulation data for Gazebo. -->
   <xacro:include filename="$(find arena-simulation-setup)/robot/jackal/urdf/jackal.gazebo" />
@@ -226,5 +262,5 @@
        of these into the final description is controlled by optenv variables, which
        default each one to off.-->
-  <xacro:include filename="$(find arena-simulation-setup)/robot/jackal/urdf/accessories.urdf.xacro" />
+  <xacro:include filename="$(find arena-simulation-setup)/robot/jackal/urdf/accessories.urdf.xacro"  />
   <!-- Optional custom includes. -->
   <xacro:include filename="$(optenv JACKAL_URDF_EXTRAS empty.urdf)" />

File: robot/ridgeback/urdf/accessories/hokuyo_ust-10lx_mount.urdf.xacro (robot description, xacro)
@@ -57,7 +57,8 @@
         </ray>
         <plugin name="gazebo_ros_laser" filename="libgazebo_ros_laser.so">
-          <topicName>${topic}</topicName>
-          <frameName>${prefix}_laser</frameName>
-          <hokuyoMinIntensity>101</hokuyoMinIntensity>
+            <topicName>${topic}</topicName>
+            <frameName>${robot_namespace}_base_footprint</frameName>
+            <tf_prefix>${robot_namespace}</tf_prefix>
+            <robotNamespace>${robot_namespace}</robotNamespace>
         </plugin>
       </sensor>

File: robot/ridgeback/urdf/ridgeback.urdf.xacro (robot description, xacro)
@@ -1,4 +1,6 @@
 <?xml version="1.0"?>
 <robot name="ridgeback" xmlns:xacro="http://ros.org/wiki/xacro">
+  <xacro:arg name="robot_namespace" default="$(optenv ROBOT_NAMESPACE /)" />
+  <xacro:property name="robot_namespace" value="$(arg robot_namespace)" />
   <xacro:property name="PI" value="3.1415926535897931" />
   <xacro:property name="wheel_radius" value="0.0759" />

File: robot/rto/urdf/components/rto_body.urdf.xacro (robot description, xacro)
@@ -57,9 +57,9 @@
         <gazebo>
             <plugin name="object_controller" filename="libgazebo_ros_planar_move.so">
-                <commandTopic>cmd_vel</commandTopic>
-                <odometryTopic>odom</odometryTopic>
-                <odometryFrame>odom</odometryFrame>
+                <commandTopic>${robot_namespace}/cmd_vel</commandTopic>
+                <odometryTopic>${robot_namespace}/odom</odometryTopic>
+                <odometryFrame>${robot_namespace}_odom</odometryFrame>
                 <odometryRate>20</odometryRate>
-                <robotBaseFrame>base_link</robotBaseFrame>
+                <robotBaseFrame>${robot_namespace}_base_footprint</robotBaseFrame>
                 <publishTF>true</publishTF>
             </plugin>

File: robot/rto/urdf/rto.urdf.xacro (robot description, xacro)
@@ -1,4 +1,6 @@
 <?xml version="1.0"?>
 <robot name="rto" xmlns:xacro="http://wiki.ros.org/xacro">
+	<xacro:arg name="robot_namespace" default="$(optenv ROBOT_NAMESPACE /)" />
+	<xacro:property name="robot_namespace" value="$(arg robot_namespace)" />
   <xacro:include filename="$(find arena-simulation-setup)/robot/rto/urdf/components/rto_parts.urdf.xacro"/>
   <xacro:include filename="$(find arena-simulation-setup)/robot/rto/urdf/components/rto_body.urdf.xacro"/>

File: robot/rto/urdf/sensors/hokuyo.urdf.xacro (robot description, xacro)
@@ -64,6 +64,8 @@
         </ray>
         <plugin name="gazebo_ros_${name}_controller" filename="libgazebo_ros_laser.so">
-          <topicName>${ros_topic}</topicName>
-          <frameName>${name}_link</frameName>
+            <topicName>${robot_namespace}/scan</topicName>
+            <frameName>${robot_namespace}_base_footprint</frameName>
+            <tf_prefix>${robot_namespace}</tf_prefix>
+            <robotNamespace>${robot_namespace}</robotNamespace>
         </plugin>
       </sensor>

File: robot/tiago/urdf/tiago.urdf.xacro (robot description, xacro)
@@ -14,4 +14,6 @@
 <robot  xmlns:xacro="http://ros.org/wiki/xacro"
         name="tiago" >
+    <xacro:arg name="robot_namespace" default="$(optenv ROBOT_NAMESPACE /)" />
+	  <xacro:property name="robot_namespace" value="$(arg robot_namespace)" />
     <xacro:arg name="arm" default="false"/> <!-- true, false -->
     <xacro:arg name="wrist_model" default="wrist-2010"/>
