Commit message: added go1 correctly

File: robot/go1/urdf/depthCamera.xacro (robot description, xacro)
@@ -17,5 +17,5 @@
                 <origin xyz="0 0 0" rpy="0 0 0"/>
                 <geometry>
-                    <mesh filename="package://go1_description/meshes/depthCamera.dae" scale="1 1 1"/>
+                    <mesh filename="package://arena-simulation-setup/robot/go1/meshes/depthCamera.dae" scale="1 1 1"/>
                 </geometry>
             </visual>

File: robot/go1/urdf/go1.urdf (robot description, URDF)
Before this commit: robot go, 47 links, 46 joints
Links:
- link FL_calf: geometry collision box size=0.213 0.016 0.016; visual mesh filename=package://arena-simulation-setup/robot/go1/meshes/calf.dae scale=1 1 1
- link FL_hip: geometry collision cylinder length=0.04 radius=0.046; visual mesh filename=package://arena-simulation-setup/robot/go1/meshes/hip.dae scale=1 1 1
- link FL_thigh: geometry collision box size=0.213 0.0245 0.034; visual mesh filename=package://arena-simulation-setup/robot/go1/meshes/thigh.dae scale=1 1 1
- link FR_calf: geometry collision box size=0.213 0.016 0.016; visual mesh filename=package://arena-simulation-setup/robot/go1/meshes/calf.dae scale=1 1 1
- link FR_hip: geometry collision cylinder length=0.04 radius=0.046; visual mesh filename=package://arena-simulation-setup/robot/go1/meshes/hip.dae scale=1 1 1
- link FR_thigh: geometry collision box size=0.213 0.0245 0.034; visual mesh filename=package://arena-simulation-setup/robot/go1/meshes/thigh_mir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 scale=1 1 1
- link RL_calf: geometry collision box size=0.213 0.016 0.016; visual mesh filename=package://arena-simulation-setup/robot/go1/meshes/calf.dae scale=1 1 1
- link RL_hip: geometry collision cylinder length=0.04 radius=0.046; visual mesh filename=package://arena-simulation-setup/robot/go1/meshes/hip.dae scale=1 1 1
- link RL_thigh: geometry collision box size=0.213 0.0245 0.034; visual mesh filename=package://arena-simulation-setup/robot/go1/meshes/thigh.dae scale=1 1 1
- link RR_calf: geometry collision box size=0.213 0.016 0.016; visual mesh filename=package://arena-simulation-setup/robot/go1/meshes/calf.dae scale=1 1 1
- link RR_hip: geometry collision cylinder length=0.04 radius=0.046; visual mesh filename=package://arena-simulation-setup/robot/go1/meshes/hip.dae scale=1 1 1
- link RR_thigh: geometry collision box size=0.213 0.0245 0.034; visual mesh filename=package://arena-simulation-setup/robot/go1/meshes/thigh_mir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 scale=1 1 1
- link camera_chin: geometry collision box size=.001 .001 .001; visual mesh filename=package://arena-simulation-setup/robot/go1/meshes/depthCame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 scale=1 1 1
- link camera_face: geometry collision box size=.001 .001 .001; visual mesh filename=package://arena-simulation-setup/robot/go1/meshes/depthCame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 scale=1 1 1
- link camera_left: geometry collision box size=.001 .001 .001; visual mesh filename=package://arena-simulation-setup/robot/go1/meshes/depthCame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 scale=1 1 1
- link camera_rearDown: geometry collision box size=.001 .001 .001; visual mesh filename=package://arena-simulation-setup/robot/go1/meshes/depthCame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 scale=1 1 1
- link camera_right: geometry collision box size=.001 .001 .001; visual mesh filename=package://arena-simulation-setup/robot/go1/meshes/depthCame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 scale=1 1 1
- link trunk: geometry collision box size=0.3762 0.0935 0.114; visual mesh filename=package://arena-simulation-setup/robot/go1/meshes/trunk.dae scale=1 1 1
- link ultraSound_face: geometry collision box size=.001 .001 .001; visual mesh filename=package://arena-simulation-setup/robot/go1/meshes/ultraSoun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 scale=1 1 1
- link ultraSound_left: geometry collision box size=.001 .001 .001; visual mesh filename=package://arena-simulation-setup/robot/go1/meshes/ultraSoun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 scale=1 1 1
- link ultraSound_right: geometry collision box size=.001 .001 .001; visual mesh filename=package://arena-simulation-setup/robot/go1/meshes/ultraSoun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 scale=1 1 1

File: robot/go1/urdf/go1.urdf.xacro (robot description, xacro)
@@ -2,13 +2,13 @@
 <robot name="go1" xmlns:xacro="http://www.ros.org/wiki/xacro">
     <xacro:arg name="DEBUG" default="false"/>
-    <xacro:include filename="$(find go1_description)/xacro/const.xacro"/>
-    <xacro:include filename="$(find go1_description)/xacro/materials.xacro"/>
-    <xacro:include filename="$(find go1_description)/xacro/leg.xacro"/>
-    <!-- <xacro:include filename="$(find go1_description)/xacro/stairs.xacro"/> -->
-    <xacro:include filename="$(find go1_description)/xacro/gazebo.xacro"/>
-    <xacro:include filename="$(find go1_description)/xacro/depthCamera.xacro"/>
-    <xacro:include filename="$(find go1_description)/xacro/ultraSound.xacro"/>
+    <xacro:include filename="$(find arena-simulation-setup)/robot/go1/xacro/const.xacro"/>
+    <xacro:include filename="$(find arena-simulation-setup)/robot/go1/xacro/materials.xacro"/>
+    <xacro:include filename="$(find arena-simulation-setup)/robot/go1/xacro/leg.xacro"/>
+    <!-- <xacro:include filename="$(find arena-simulation-setup)/robot/go1/xacro/stairs.xacro"/> -->
+    <xacro:include filename="$(find arena-simulation-setup)/robot/go1/xacro/gazebo.xacro"/>
+    <xacro:include filename="$(find arena-simulation-setup)/robot/go1/xacro/depthCamera.xacro"/>
+    <xacro:include filename="$(find arena-simulation-setup)/robot/go1/xacro/ultraSound.xacro"/>
     <!-- <xacro:include filename="$(find go1_gazebo)/launch/stairs.urdf.xacro"/> -->
-    <xacro:include filename="$(find go1_description)/xacro/lidar.xacro"/>
+    <xacro:include filename="$(find arena-simulation-setup)/robot/go1/xacro/lidar.xacro"/>
     <!-- <xacro:stairs stairs="15" xpos="0" ypos="0" zpos="0" /> -->
     <!-- Rotor related joint and link is only for demonstrate location. -->
@@ -40,5 +40,5 @@
             <origin rpy="0 0 0" xyz="0 0 0"/>
             <geometry>
-                <mesh filename="package://go1_description/meshes/trunk.dae" scale="1 1 1"/>
+                <mesh filename="package://arena-simulation-setup/robot/go1/meshes/trunk.dae" scale="1 1 1"/>
             </geometry>
             <!-- <material name="orange"/> -->

File: robot/go1/urdf/leg.xacro (robot description, xacro)
@@ -1,5 +1,5 @@
 <?xml version="1.0"?>
 <robot xmlns:xacro="http://www.ros.org/wiki/xacro">
-    <xacro:include filename="$(find go1_description)/xacro/transmission.xacro"/>
+    <xacro:include filename="$(find arena-simulation-setup)/robot/go1/xacro/transmission.xacro"/>
     <xacro:macro name="leg" params="name mirror mirror_dae front_hind front_hind_dae">
         <joint name="${name}_hip_joint" type="revolute">
@@ -58,5 +58,5 @@
                 </xacro:if>
                 <geometry>
-                    <mesh filename="package://go1_description/meshes/hip.dae" scale="1 1 1"/>
+                    <mesh filename="package://arena-simulation-setup/robot/go1/meshes/hip.dae" scale="1 1 1"/>
                 </geometry>
                 <!-- <material name="orange"/> -->
@@ -118,8 +118,8 @@
                 <geometry>
                     <xacro:if value="${mirror_dae == True}">
-                        <mesh filename="package://go1_description/meshes/thigh.dae" scale="1 1 1"/>
+                        <mesh filename="package://arena-simulation-setup/robot/go1/meshes/thigh.dae" scale="1 1 1"/>
                     </xacro:if>
                     <xacro:if value="${mirror_dae == False}">
-                        <mesh filename="package://go1_description/meshes/thigh_mirror.dae" scale="1 1 1"/>
+                        <mesh filename="package://arena-simulation-setup/robot/go1/meshes/thigh_mirror.dae" scale="1 1 1"/>
                     </xacro:if>
                 </geometry>
@@ -181,5 +181,5 @@
                 <origin rpy="0 0 0" xyz="0 0 0"/>
                 <geometry>
-                    <mesh filename="package://go1_description/meshes/calf.dae" scale="1 1 1"/>
+                    <mesh filename="package://arena-simulation-setup/robot/go1/meshes/calf.dae" scale="1 1 1"/>
                 </geometry>
                 <!-- <material name="orange"/> -->

File: robot/go1/urdf/ultraSound.xacro (robot description, xacro)
@@ -17,5 +17,5 @@
             <origin xyz="0 0 0" rpy="0 0 0"/>
             <geometry>
-                <mesh filename="package://go1_description/meshes/ultraSound.dae" scale="1 1 1"/>
+                <mesh filename="package://arena-simulation-setup/robot/go1/meshes/ultraSound.dae" scale="1 1 1"/>
             </geometry>
             <material name="black"/>

File: robot/go1/xacro/gazebo.xacro (robot description, xacro)
@@ -4,6 +4,5 @@
     <gazebo>
         <plugin name="gazebo_ros_control" filename="libgazebo_ros_control.so">
-            <robotNamespace>go1_gazebo</robotNamespace>
-            <robotSimType>gazebo_ros_control/DefaultRobotHWSim</robotSimType>
+            <!-- <robotSimType>gazebo_ros_control/DefaultRobotHWSim</robotSimType> -->
         </plugin>
     </gazebo>

File: robot/go1/xacro/robot.xacro (robot description, xacro)
@@ -2,13 +2,13 @@
 <robot name="go1" xmlns:xacro="http://www.ros.org/wiki/xacro">
     <xacro:arg name="DEBUG" default="false"/>
-    <xacro:include filename="$(find go1_description)/xacro/const.xacro"/>
-    <xacro:include filename="$(find go1_description)/xacro/materials.xacro"/>
-    <xacro:include filename="$(find go1_description)/xacro/leg.xacro"/>
-    <!-- <xacro:include filename="$(find go1_description)/xacro/stairs.xacro"/> -->
-    <xacro:include filename="$(find go1_description)/xacro/gazebo.xacro"/>
-    <xacro:include filename="$(find go1_description)/xacro/depthCamera.xacro"/>
-    <xacro:include filename="$(find go1_description)/xacro/ultraSound.xacro"/>
+    <xacro:include filename="$(find arena-simulation-setup/robot/go1/xacro/const.xacro"/>
+    <xacro:include filename="$(find arena-simulation-setup/robot/go1/xacro/materials.xacro"/>
+    <xacro:include filename="$(find arena-simulation-setup/robot/go1/xacro/leg.xacro"/>
+    <!-- <xacro:include filename="$(find arena-simulation-setup/robot/go1/xacro/stairs.xacro"/> -->
+    <xacro:include filename="$(find arena-simulation-setup/robot/go1/xacro/gazebo.xacro"/>
+    <xacro:include filename="$(find arena-simulation-setup/robot/go1/xacro/depthCamera.xacro"/>
+    <xacro:include filename="$(find arena-simulation-setup/robot/go1/xacro/ultraSound.xacro"/>
     <!-- <xacro:include filename="$(find go1_gazebo)/launch/stairs.urdf.xacro"/> -->
-    <xacro:include filename="$(find go1_description)/xacro/lidar.xacro"/>
+    <xacro:include filename="$(find arena-simulation-setup/robot/go1/xacro/lidar.xacro"/>
     <!-- <xacro:stairs stairs="15" xpos="0" ypos="0" zpos="0" /> -->
     <!-- Rotor related joint and link is only for demonstrate location. -->
@@ -40,5 +40,5 @@
             <origin rpy="0 0 0" xyz="0 0 0"/>
             <geometry>
-                <mesh filename="package://go1_description/meshes/trunk.dae" scale="1 1 1"/>
+                <mesh filename="package://arena-simulation-setup/robot/go1/meshes/trunk.dae" scale="1 1 1"/>
             </geometry>
             <!-- <material name="orange"/> -->
