Commit message: init go1

File: robot/go1/urdf/go1.urdf (robot description, URDF)
Before this commit: robot go1, 47 links, 46 joints
Links:
- link FL_calf: geometry collision box size=0.213 0.016 0.016; visual mesh filename=package://arena-simulation-setup/robot/go1/meshes/calf.dae scale=1 1 1
- link FL_hip: geometry collision cylinder length=0.04 radius=0.046; visual mesh filename=package://arena-simulation-setup/robot/go1/meshes/hip.dae scale=1 1 1
- link FL_thigh: geometry collision box size=0.213 0.0245 0.034; visual mesh filename=package://arena-simulation-setup/robot/go1/meshes/thigh.dae scale=1 1 1
- link FR_calf: geometry collision box size=0.213 0.016 0.016; visual mesh filename=package://arena-simulation-setup/robot/go1/meshes/calf.dae scale=1 1 1
- link FR_hip: geometry collision cylinder length=0.04 radius=0.046; visual mesh filename=package://arena-simulation-setup/robot/go1/meshes/hip.dae scale=1 1 1
- link FR_thigh: geometry collision box size=0.213 0.0245 0.034; visual mesh filename=package://arena-simulation-setup/robot/go1/meshes/thigh_mir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 scale=1 1 1
- link RL_calf: geometry collision box size=0.213 0.016 0.016; visual mesh filename=package://arena-simulation-setup/robot/go1/meshes/calf.dae scale=1 1 1
- link RL_hip: geometry collision cylinder length=0.04 radius=0.046; visual mesh filename=package://arena-simulation-setup/robot/go1/meshes/hip.dae scale=1 1 1
- link RL_thigh: geometry collision box size=0.213 0.0245 0.034; visual mesh filename=package://arena-simulation-setup/robot/go1/meshes/thigh.dae scale=1 1 1
- link RR_calf: geometry collision box size=0.213 0.016 0.016; visual mesh filename=package://arena-simulation-setup/robot/go1/meshes/calf.dae scale=1 1 1
- link RR_hip: geometry collision cylinder length=0.04 radius=0.046; visual mesh filename=package://arena-simulation-setup/robot/go1/meshes/hip.dae scale=1 1 1
- link RR_thigh: geometry collision box size=0.213 0.0245 0.034; visual mesh filename=package://arena-simulation-setup/robot/go1/meshes/thigh_mir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 scale=1 1 1
- link camera_chin: geometry collision box size=.001 .001 .001; visual mesh filename=package://arena-simulation-setup/robot/go1/meshes/depthCame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 scale=1 1 1
- link camera_face: geometry collision box size=.001 .001 .001; visual mesh filename=package://arena-simulation-setup/robot/go1/meshes/depthCame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 scale=1 1 1
- link camera_left: geometry collision box size=.001 .001 .001; visual mesh filename=package://arena-simulation-setup/robot/go1/meshes/depthCame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 scale=1 1 1
- link camera_rearDown: geometry collision box size=.001 .001 .001; visual mesh filename=package://arena-simulation-setup/robot/go1/meshes/depthCame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 scale=1 1 1
- link camera_right: geometry collision box size=.001 .001 .001; visual mesh filename=package://arena-simulation-setup/robot/go1/meshes/depthCame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 scale=1 1 1
- link trunk: geometry collision box size=0.3762 0.0935 0.114; visual mesh filename=package://arena-simulation-setup/robot/go1/meshes/trunk.dae scale=1 1 1
- link ultraSound_face: geometry collision box size=.001 .001 .001; visual mesh filename=package://arena-simulation-setup/robot/go1/meshes/ultraSoun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 scale=1 1 1
- link ultraSound_left: geometry collision box size=.001 .001 .001; visual mesh filename=package://arena-simulation-setup/robot/go1/meshes/ultraSoun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 scale=1 1 1
- link ultraSound_right: geometry collision box size=.001 .001 .001; visual mesh filename=package://arena-simulation-setup/robot/go1/meshes/ultraSoun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 scale=1 1 1
