Commit message: implement inetrial_link

File: robot/buddy/xacro/gazebo.xacro (robot description, xacro)
@@ -29,9 +29,29 @@
     </gazebo>
     <gazebo reference="rear_caster_caster_wheel">
-			<mu1 value="0.0001"/>
-			<mu2 value="0.0001"/>
-			<kp value="10000000.0" />
-			<kd value="1.0" />
-			<fdir1 value="1 0 0"/>
-		</gazebo>
+        <mu1 value="0.0001"/>
+        <mu2 value="0.0001"/>
+        <kp value="10000000.0" />
+        <kd value="1.0" />
+        <fdir1 value="1 0 0"/>
+    </gazebo>
+    <gazebo reference="inertial_link">
+        <gravity>true</gravity>
+        <sensor name="imu_sensor" type="imu">
+            <always_on>true</always_on>
+            <update_rate>100</update_rate>
+            <visualize>true</visualize>
+            <topic>imu/data</topic>
+            <plugin filename="libgazebo_ros_imu_sensor.so" name="imu_plugin">
+                <topicName>imu</topicName>
+                <bodyName>inertial_link</bodyName>
+                <updateRateHZ>10.0</updateRateHZ>
+                <gaussianNoise>0.0</gaussianNoise>
+                <xyzOffset>0 0 0</xyzOffset>
+                <rpyOffset>0 0 0</rpyOffset>
+                <frameName>buddy_0_0/inertial_link</frameName>
+                <initialOrientationAsReference>false</initialOrientationAsReference>
+            </plugin>
+            <pose>0 0 0 0 0 0</pose>
+        </sensor>
+    </gazebo>
 </robot>

File: robot/buddy/xacro/robot.xacro (robot description, xacro)
@@ -30,10 +30,10 @@
     </link>
     <joint name="inertial_joint" type="fixed">
-            <origin rpy="0 0 0" xyz="0 0 0"/>
-            <parent link="base_link"/>
-            <child link="inertial_link"/>
+        <origin rpy="0 0 0" xyz="0 0 0"/>
+        <parent link="base_link"/>
+        <child link="inertial_link"/>
     </joint>
     <link name="inertial_link">
-     <inertial>
+        <inertial>
             <origin rpy="0 0 0" xyz="${chassis_com_x} ${chassis_com_y} ${chassis_com_z}"/>
             <mass value="${chassis_mass}"/>
