Commit message: fixed 2d lidar + cameras

File: robot/buddy/xacro/const.xacro (robot description, xacro)
@@ -4,5 +4,5 @@
     <!--  3DLIDAR -->
     <xacro:property name="helios_com_x" value="0.1091"/>
-    <xacro:property name="helios_com_z" value="1.091"/>
+    <xacro:property name="helios_com_z" value="0.951"/>
     <!-- rotation in degrees  -->
     <xacro:property name="helios_pitch" value="10.0"/>
