Commit message: prepare for production

File: robot/buddy/urdf/buddy.urdf.xacro (robot description, xacro)
@@ -6,17 +6,17 @@
     <xacro:arg name="ip_cameras_enabled" default="false" />
     <!-- <xacro:arg name="robot_namespace" default="/" /> -->
-    <xacro:include filename="$(find buddy_description)/xacro/const.xacro"/>
-    <xacro:include filename="$(find buddy_description)/xacro/wheel.xacro"/>
-    <xacro:include filename="$(find buddy_description)/xacro/gazebo.xacro"/>
-    <xacro:include filename="$(find buddy_description)/xacro/gazebo_rgbd.xacro"/>
-    <xacro:include filename="$(find buddy_description)/xacro/gazebo_camera.xacro"/>
-    <xacro:include filename="$(find buddy_description)/xacro/sick_scan.urdf.xacro"/>
+    <xacro:include filename="$(find arena-simulation-setup)/robot/buddy/xacro/const.xacro"/>
+    <xacro:include filename="$(find arena-simulation-setup)/robot/buddy/xacro/wheel.xacro"/>
+    <xacro:include filename="$(find arena-simulation-setup)/robot/buddy/xacro/gazebo.xacro"/>
+    <xacro:include filename="$(find arena-simulation-setup)/robot/buddy/xacro/gazebo_rgbd.xacro"/>
+    <xacro:include filename="$(find arena-simulation-setup)/robot/buddy/xacro/gazebo_camera.xacro"/>
+    <xacro:include filename="$(find arena-simulation-setup)/robot/buddy/xacro/sick_scan.urdf.xacro"/>
     <xacro:include filename="$(find velodyne_description)/urdf/VLP-16.urdf.xacro"/>
-    <xacro:include filename="$(find buddy_description)/xacro/VLP-1.urdf.xacro"/>
+    <xacro:include filename="$(find arena-simulation-setup)/robot/buddy/xacro/VLP-1.urdf.xacro"/>
     <!-- Robot Base -->
     <link name="base_link">
         <visual>
             <geometry>
-                <mesh filename="package://buddy_description/meshes/buddy_simplified_mesh.stl" scale="1 1 1 "/>
+                <mesh filename="package://arena-simulation-setup/robot/buddy/meshes/buddy_simplified_mesh.stl" scale="1 1 1 "/>
             </geometry>
         </visual>
@@ -25,5 +25,5 @@
             <origin rpy="0 0 0" xyz="0 0 0"/>
             <geometry>
-                <mesh filename="package://buddy_description/meshes/buddy_simplified_mesh.stl" scale="1 1 1 "/>
+                <mesh filename="package://arena-simulation-setup/robot/buddy/meshes/buddy_simplified_mesh.stl" scale="1 1 1 "/>
             </geometry>
         </collision>

File: robot/buddy/urdf/wheel.xacro (robot description, xacro)
@@ -1,5 +1,5 @@
 <?xml version="1.0"?>
 <robot xmlns:xacro="http://www.ros.org/wiki/xacro">
-    <xacro:include filename="$(find buddy_description)/xacro/transmission.xacro"/>
+    <xacro:include filename="$(find arena-simulation-setup)/robot/buddy/xacro/transmission.xacro"/>
     <xacro:macro name="wheel" params="name *origin">
         <joint name="${name}_wheel_joint" type="continuous">

File: robot/buddy/xacro/robot.xacro (robot description, xacro)
@@ -1,22 +1,22 @@
 <?xml version="1.0"?>
 <robot name="buddy" xmlns:xacro="http://www.ros.org/wiki/xacro">
-    <xacro:arg name="helios_5515_enabled" default="false" />
+    <xacro:arg name="helios_5515_enabled" default="true" />
     <xacro:arg name="helios_1_enabled" default="false" />
-    <xacro:arg name="rgbd_enabled" default="false" />
-    <xacro:arg name="ip_cameras_enabled" default="false" />
+    <xacro:arg name="rgbd_enabled" default="true" />
+    <xacro:arg name="ip_cameras_enabled" default="true" />
     <!-- <xacro:arg name="robot_namespace" default="/" /> -->
-    <xacro:include filename="$(find buddy_description)/xacro/const.xacro"/>
-    <xacro:include filename="$(find buddy_description)/xacro/wheel.xacro"/>
-    <xacro:include filename="$(find buddy_description)/xacro/gazebo.xacro"/>
-    <xacro:include filename="$(find buddy_description)/xacro/gazebo_rgbd.xacro"/>
-    <xacro:include filename="$(find buddy_description)/xacro/gazebo_camera.xacro"/>
-    <xacro:include filename="$(find buddy_description)/xacro/sick_scan.urdf.xacro"/>
+    <xacro:include filename="$(find arena-simulation-setup)/robot/buddy/xacro/const.xacro"/>
+    <xacro:include filename="$(find arena-simulation-setup)/robot/buddy/xacro/wheel.xacro"/>
+    <xacro:include filename="$(find arena-simulation-setup)/robot/buddy/xacro/gazebo.xacro"/>
+    <xacro:include filename="$(find arena-simulation-setup)/robot/buddy/xacro/gazebo_rgbd.xacro"/>
+    <xacro:include filename="$(find arena-simulation-setup)/robot/buddy/xacro/gazebo_camera.xacro"/>
+    <xacro:include filename="$(find arena-simulation-setup)/robot/buddy/xacro/sick_scan.urdf.xacro"/>
     <xacro:include filename="$(find velodyne_description)/urdf/VLP-16.urdf.xacro"/>
-    <xacro:include filename="$(find buddy_description)/xacro/VLP-1.urdf.xacro"/>
+    <xacro:include filename="$(find arena-simulation-setup)/robot/buddy/xacro/VLP-1.urdf.xacro"/>
     <!-- Robot Base -->
     <link name="base_link">
         <visual>
             <geometry>
-                <mesh filename="package://buddy_description/meshes/buddy_simplified_mesh.stl" scale="1 1 1 "/>
+                <mesh filename="package://arena-simulation-setup/robot/buddy/meshes/buddy_simplified_mesh.stl" scale="1 1 1 "/>
             </geometry>
         </visual>
@@ -25,5 +25,5 @@
             <origin rpy="0 0 0" xyz="0 0 0"/>
             <geometry>
-                <mesh filename="package://buddy_description/meshes/buddy_simplified_mesh.stl" scale="1 1 1 "/>
+                <mesh filename="package://arena-simulation-setup/robot/buddy/meshes/buddy_simplified_mesh.stl" scale="1 1 1 "/>
             </geometry>
         </collision>
