Commit message: Fixes for launch files

File: robot/waffle/urdf/waffle.urdf.xacro (robot description, xacro)
@@ -1,4 +1,4 @@
 <?xml version="1.0" ?>
-<robot name="turtlebot3_waffle_pi" xmlns:xacro="http://ros.org/wiki/xacro">
+<robot name="waffle" xmlns:xacro="http://ros.org/wiki/xacro">
   <xacro:include filename="$(find arena-simulation-setup)/robot/waffle/urdf/common_properties.xacro"/>
   <xacro:include filename="$(find arena-simulation-setup)/robot/waffle/urdf/waffle.gazebo.xacro"/>
@@ -13,5 +13,5 @@
       <origin xyz="-0.064 0 0.0" rpy="0 0 0"/>
       <geometry>
-        <mesh filename="package://arena-simulation-setup/robot/turtlebot3_waffle_pi/meshes/bases/waffle_pi_base.stl" scale="0.001 0.001 0.001"/>
+        <mesh filename="package://arena-simulation-setup/robot/waffle/meshes/bases/waffle_pi_base.stl" scale="0.001 0.001 0.001"/>
       </geometry>
       <material name="light_black"/>
@@ -41,5 +41,5 @@
       <origin xyz="0 0 0" rpy="1.57 0 0"/>
       <geometry>
-        <mesh filename="package://arena-simulation-setup/robot/turtlebot3_waffle_pi/meshes/wheels/left_tire.stl" scale="0.001 0.001 0.001"/>
+        <mesh filename="package://arena-simulation-setup/robot/waffle/meshes/wheels/left_tire.stl" scale="0.001 0.001 0.001"/>
       </geometry>
       <material name="dark"/>
@@ -69,5 +69,5 @@
       <origin xyz="0 0 0" rpy="1.57 0 0"/>
       <geometry>
-        <mesh filename="package://arena-simulation-setup/robot/turtlebot3_waffle_pi/meshes/wheels/right_tire.stl" scale="0.001 0.001 0.001"/>
+        <mesh filename="package://arena-simulation-setup/robot/waffle/meshes/wheels/right_tire.stl" scale="0.001 0.001 0.001"/>
       </geometry>
       <material name="dark"/>
@@ -142,5 +142,5 @@
       <origin xyz="0 0 0.0" rpy="0 0 0"/>
       <geometry>
-        <mesh filename="package://arena-simulation-setup/robot/turtlebot3_waffle_pi/meshes/sensors/lds.stl" scale="0.001 0.001 0.001"/>
+        <mesh filename="package://arena-simulation-setup/robot/waffle/meshes/sensors/lds.stl" scale="0.001 0.001 0.001"/>
       </geometry>
       <material name="dark"/>

Commit message: fix waffle

File: robot/waffle/urdf/waffle.urdf.xacro (robot description, xacro)
@@ -15,5 +15,5 @@
       <origin xyz="-0.064 0 0.0" rpy="0 0 0"/>
       <geometry>
-        <mesh filename="package://arena-simulation-setup/robot/waffle/meshes/bases/waffle_pi_base.stl" scale="0.001 0.001 0.001"/>
+        <mesh filename="package://arena-simulation-setup/robot/waffle/urdf/meshes/bases/waffle_pi_base.stl" scale="0.001 0.001 0.001"/>
       </geometry>
       <material name="light_black"/>
@@ -43,5 +43,5 @@
       <origin xyz="0 0 0" rpy="1.57 0 0"/>
       <geometry>
-        <mesh filename="package://arena-simulation-setup/robot/waffle/meshes/wheels/left_tire.stl" scale="0.001 0.001 0.001"/>
+        <mesh filename="package://arena-simulation-setup/robot/waffle/urdf/meshes/wheels/left_tire.stl" scale="0.001 0.001 0.001"/>
       </geometry>
       <material name="dark"/>
@@ -71,5 +71,5 @@
       <origin xyz="0 0 0" rpy="1.57 0 0"/>
       <geometry>
-        <mesh filename="package://arena-simulation-setup/robot/waffle/meshes/wheels/right_tire.stl" scale="0.001 0.001 0.001"/>
+        <mesh filename="package://arena-simulation-setup/robot/waffle/urdf/meshes/wheels/right_tire.stl" scale="0.001 0.001 0.001"/>
       </geometry>
       <material name="dark"/>
@@ -144,5 +144,5 @@
       <origin xyz="0 0 0.0" rpy="0 0 0"/>
       <geometry>
-        <mesh filename="package://arena-simulation-setup/robot/waffle/meshes/sensors/lds.stl" scale="0.001 0.001 0.001"/>
+        <mesh filename="package://arena-simulation-setup/robot/waffle/urdf/meshes/sensors/lds.stl" scale="0.001 0.001 0.001"/>
       </geometry>
       <material name="dark"/>
