Commit message: cleanup

File: robot/dingo/urdf/accessories/hokuyo_ust10.urdf.xacro (robot description, xacro)
@@ -53,5 +53,5 @@
         <geometry>
           <!-- Origin of this mesh is the base of the bracket. -->
-          <mesh filename="package://arena-simulation-setup/robot/dingo/meshes/hokuyo_ust10.stl" />
+          <mesh filename="package://arena-simulation-setup/robot/dingo/urdf/meshes/hokuyo_ust10.stl" />
         </geometry>
         <material name="dark_grey" />

File: robot/dingo/urdf/accessories/sick_lms1xx_mount.urdf.xacro (robot description, xacro)
@@ -34,5 +34,5 @@
         <geometry>
           <!-- Origin of this mesh is the base of the bracket. -->
-          <mesh filename="package://arena-simulation-setup/robot/dingo/meshes/sick-lms1xx-bracket.stl" />
+          <mesh filename="package://arena-simulation-setup/robot/dingo/urdf/meshes/sick-lms1xx-bracket.stl" />
         </geometry>
         <material name="dark_grey" />

File: robot/dingo/urdf/dingo-d.urdf.xacro (robot description, xacro)
@@ -18,5 +18,5 @@
         <origin xyz="0 0 0" rpy="0 0 0"/>
         <geometry>
-          <mesh filename="package://arena-simulation-setup/robot/dingo/meshes/wheel.stl"/>
+          <mesh filename="package://arena-simulation-setup/robot/dingo/urdf/meshes/wheel.stl"/>
         </geometry>
         <material name="black" />
@@ -125,5 +125,5 @@
       <origin xyz="0 0 0" rpy="0 0 0"/>
       <geometry>
-        <mesh filename="package://arena-simulation-setup/robot/dingo/meshes/diff_chassis.dae"/>
+        <mesh filename="package://arena-simulation-setup/robot/dingo/urdf/meshes/diff_chassis.dae"/>
       </geometry>
     </visual>
@@ -131,5 +131,5 @@
       <origin xyz="0 0 0"/>
       <geometry>
-        <mesh filename="package://arena-simulation-setup/robot/dingo/meshes/diff_chassis_collision.stl"/>
+        <mesh filename="package://arena-simulation-setup/robot/dingo/urdf/meshes/diff_chassis_collision.stl"/>
       </geometry>
     </collision>

File: robot/dingo/urdf/dingo.urdf.xacro (robot description, xacro)
@@ -19,5 +19,5 @@
         <origin xyz="0 0 0" rpy="0 0 0"/>
         <geometry>
-          <mesh filename="package://arena-simulation-setup/robot/dingo/meshes/wheel.stl"/>
+          <mesh filename="package://arena-simulation-setup/robot/dingo/urdf/meshes/wheel.stl"/>
         </geometry>
         <material name="black" />
@@ -126,5 +126,5 @@
       <origin xyz="0 0 0" rpy="0 0 0"/>
       <geometry>
-        <mesh filename="package://arena-simulation-setup/robot/dingo/meshes/diff_chassis.dae"/>
+        <mesh filename="package://arena-simulation-setup/robot/dingo/urdf/meshes/diff_chassis.dae"/>
       </geometry>
     </visual>
@@ -132,5 +132,5 @@
       <origin xyz="0 0 0"/>
       <geometry>
-        <mesh filename="package://arena-simulation-setup/robot/dingo/meshes/diff_chassis_collision.stl"/>
+        <mesh filename="package://arena-simulation-setup/robot/dingo/urdf/meshes/diff_chassis_collision.stl"/>
       </geometry>
     </collision>
