Commit message: cleanup

File: robot/jackal/urdf/accessories.urdf.xacro (robot description, xacro)
@@ -153,5 +153,5 @@
         <origin xyz="0 0 0" rpy="0 0 0"/>
         <geometry>
-          <mesh filename="package://jackal_description/meshes/ark_enclosure.stl"/>
+          <mesh filename="package://jackal_description/urdf/meshes/ark_enclosure.stl"/>
         </geometry>
         <material name="dark_grey" />

File: robot/jackal/urdf/accessories/bridge_plate.urdf.xacro (robot description, xacro)
@@ -11,5 +11,5 @@
         <origin xyz="0 0 0" rpy="1.5707 0.0 1.5707" />
         <geometry>
-          <mesh filename="package://arena-simulation-setup/robot/jackal/meshes/bridge-plate.stl"/>
+          <mesh filename="package://arena-simulation-setup/robot/jackal/urdf/meshes/bridge-plate.stl"/>
         </geometry>
         <material name="dark_grey" />

File: robot/jackal/urdf/accessories/camera_mount.urdf.xacro (robot description, xacro)
@@ -5,5 +5,5 @@
         <origin xyz="0 0 0" rpy="1.5707 0 1.5707" />
         <geometry>
-          <mesh filename="package://arena-simulation-setup/robot/jackal/meshes/camera-bracket.stl" scale="0.001 0.001 0.001" />
+          <mesh filename="package://arena-simulation-setup/robot/jackal/urdf/meshes/camera-bracket.stl" scale="0.001 0.001 0.001" />
         </geometry>
         <material name="dark_grey" />
@@ -14,5 +14,5 @@
         <origin xyz="0 0 0" rpy="0 0 1.5707" />
         <geometry>
-          <mesh filename="package://arena-simulation-setup/robot/jackal/meshes/camera-beam.stl" scale="0.001 0.001 0.001" />
+          <mesh filename="package://arena-simulation-setup/robot/jackal/urdf/meshes/camera-beam.stl" scale="0.001 0.001 0.001" />
         </geometry>
         <material name="dark_grey" />

File: robot/jackal/urdf/accessories/hokuyo_ust10.urdf.xacro (robot description, xacro)
@@ -55,5 +55,5 @@
         <geometry>
           <!-- Origin of this mesh is the base of the bracket. -->
-          <mesh filename="package://arena-simulation-setup/robot/jackal/meshes/hokuyo_ust10.stl" />
+          <mesh filename="package://arena-simulation-setup/robot/jackal/urdf/meshes/hokuyo_ust10.stl" />
         </geometry>
         <material name="dark_grey" />

File: robot/jackal/urdf/accessories/novatel_smart6.urdf.xacro (robot description, xacro)
@@ -6,5 +6,5 @@
       <origin xyz="0 0 0" rpy="0 0 0" />
       <geometry>
-        <mesh filename="package://arena-simulation-setup/robot/jackal/meshes/novatel-smart6.stl"/>
+        <mesh filename="package://arena-simulation-setup/robot/jackal/urdf/meshes/novatel-smart6.stl"/>
       </geometry>
       <material name="novatel_white">

File: robot/jackal/urdf/accessories/sick_lms1xx_mount.urdf.xacro (robot description, xacro)
@@ -39,5 +39,5 @@
         <geometry>
           <!-- Origin of this mesh is the base of the bracket. -->
-          <mesh filename="package://arena-simulation-setup/robot/jackal/meshes/sick-lms1xx-bracket.stl" />
+          <mesh filename="package://arena-simulation-setup/robot/jackal/urdf/meshes/sick-lms1xx-bracket.stl" />
         </geometry>
         <material name="dark_grey" />

File: robot/jackal/urdf/accessories/stereo_camera_mount.urdf.xacro (robot description, xacro)
@@ -6,5 +6,5 @@
         <origin xyz="0 0 0" rpy="0 0 0" />
         <geometry>
-          <mesh filename="package://arena-simulation-setup/robot/jackal/meshes/stereo-camera-bracket.stl" />
+          <mesh filename="package://arena-simulation-setup/robot/jackal/urdf/meshes/stereo-camera-bracket.stl" />
         </geometry>
         <material name="dark_grey" />
@@ -15,5 +15,5 @@
         <origin xyz="0 0 0" rpy="0 0 0" />
         <geometry>
-          <mesh filename="package://arena-simulation-setup/robot/jackal/meshes/stereo-camera-beam.stl" />
+          <mesh filename="package://arena-simulation-setup/robot/jackal/urdf/meshes/stereo-camera-beam.stl" />
         </geometry>
         <material name="dark_grey" />

File: robot/jackal/urdf/jackal.urdf (robot description, URDF)
Before this commit: robot jackal, 15 links, 14 joints
Links:
- link chassis_link: geometry collision box size=0.42 0.31 0.184; visual mesh filename=package://arena-simulation-setup/robot/jackal/urdf/meshes/j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
- link front_fender_link: geometry visual mesh filename=package://arena-simulation-setup/robot/jackal/urdf/meshes/j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
- link front_laser_mount: geometry visual mesh filename=package://arena-simulation-setup/robot/jackal/urdf/meshes/h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
- link front_left_wheel_link: geometry collision cylinder length=0.04 radius=0.098; visual mesh filename=package://arena-simulation-setup/robot/jackal/urdf/meshes/j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
- link front_right_wheel_link: geometry collision cylinder length=0.04 radius=0.098; visual mesh filename=package://arena-simulation-setup/robot/jackal/urdf/meshes/j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
- link rear_fender_link: geometry visual mesh filename=package://arena-simulation-setup/robot/jackal/urdf/meshes/j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
- link rear_left_wheel_link: geometry collision cylinder length=0.04 radius=0.098; visual mesh filename=package://arena-simulation-setup/robot/jackal/urdf/meshes/j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
- link rear_right_wheel_link: geometry collision cylinder length=0.04 radius=0.098; visual mesh filename=package://arena-simulation-setup/robot/jackal/urdf/meshes/j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

File: robot/jackal/urdf/jackal.urdf.xacro (robot description, xacro)
@@ -22,5 +22,5 @@
         <origin xyz="0 0 0" rpy="${PI/2} 0 0"/>
         <geometry>
-          <mesh filename="package://arena-simulation-setup/robot/jackal/meshes/jackal-wheel.stl"/>
+          <mesh filename="package://arena-simulation-setup/robot/jackal/urdf/meshes/jackal-wheel.stl"/>
         </geometry>
         <material name="black" />
@@ -90,5 +90,5 @@
       <origin xyz="0 0 ${footprint_vertical_offset}" rpy="${PI/2} 0 ${PI/2}"/>
       <geometry>
-        <mesh filename="package://arena-simulation-setup/robot/jackal/meshes/jackal-base.stl"/>
+        <mesh filename="package://arena-simulation-setup/robot/jackal/urdf/meshes/jackal-base.stl"/>
       </geometry>
       <material name="dark_grey" />
@@ -115,5 +115,5 @@
       <visual>
         <geometry>
-          <mesh filename="package://arena-simulation-setup/robot/jackal/meshes/jackal-fender.stl"/>
+          <mesh filename="package://arena-simulation-setup/robot/jackal/urdf/meshes/jackal-fender.stl"/>
         </geometry>
         <material name="yellow" />
@@ -125,5 +125,5 @@
       <visual>
         <geometry>
-          <mesh filename="package://arena-simulation-setup/robot/jackal/meshes/accessory_fender.stl"/>
+          <mesh filename="package://arena-simulation-setup/robot/jackal/urdf/meshes/accessory_fender.stl"/>
         </geometry>
         <material name="yellow" />
@@ -146,5 +146,5 @@
       <visual>
         <geometry>
-          <mesh filename="package://arena-simulation-setup/robot/jackal/meshes/jackal-fender.stl"/>
+          <mesh filename="package://arena-simulation-setup/robot/jackal/urdf/meshes/jackal-fender.stl"/>
         </geometry>
         <material name="yellow" />
@@ -156,5 +156,5 @@
       <visual>
         <geometry>
-          <mesh filename="package://arena-simulation-setup/robot/jackal/meshes/accessory_fender.stl"/>
+          <mesh filename="package://arena-simulation-setup/robot/jackal/urdf/meshes/accessory_fender.stl"/>
         </geometry>
         <material name="yellow" />

Commit message: jackal coordinate change

File: robot/jackal/urdf/accessories.urdf.xacro (robot description, xacro)
@@ -19,6 +19,6 @@
     Add primary/secondary 2D lidar sensors.  By default these are SICK LMS1xx but can be changed with the
     JACKAL_LASER_MODEL and JACKAL_LASER_SECONDARY_MODEL environment variables. Valid model designations are:
-    - lms1xx (default) :: SICK LMS1xx
-    - ust10            :: Hokuyo UST10
+    - lms1xx           :: SICK LMS1xx
+    - ust10  (default) :: Hokuyo UST10
   -->
   <xacro:if value="$(optenv JACKAL_LASER 1)">

File: robot/jackal/urdf/jackal.urdf.xacro (robot description, xacro)
@@ -213,5 +213,5 @@
     <parent link="mid_mount" />
     <child link="rear_mount" />
-    <origin xyz="${-mount_spacing} 0 0" />
+    <origin xyz="${mount_spacing} 0 0" />
   </joint>
   <link name="front_mount"></link>
@@ -219,5 +219,5 @@
     <parent link="mid_mount" />
     <child link="front_mount" />
-    <origin xyz="${mount_spacing} 0 0" />
+    <origin xyz="${-mount_spacing} 0 0" rpy="0 0 3.14159" />
   </joint>
   <!-- Bring in simulation data for Gazebo. -->
