Commit message: mbf-teb-jackal

File: robot/jackal/urdf/jackal.urdf.xacro (robot description, xacro)
@@ -80,8 +80,8 @@
     <origin xyz="${-wheelbase/2} ${-track/2} ${wheel_vertical_offset}" rpy="0 0 0" />
   </xacro:wheel>
-  <link name="base_link"></link>
-  <joint name="base_link_joint" type="fixed">
+  <link name="link_base"></link>
+  <joint name="link_base_joint" type="fixed">
     <origin xyz="0 0 0" rpy="0 0 0" />
-    <parent link="base_link"/>
+    <parent link="link_base"/>
     <child link="chassis_link" />
   </joint>

Commit message: cleanup

File: robot/jackal/urdf/jackal.urdf.xacro (robot description, xacro)
@@ -219,5 +219,5 @@
     <parent link="mid_mount" />
     <child link="front_mount" />
-    <origin xyz="${-mount_spacing} 0 0" rpy="0 0 3.14159" />
+    <origin xyz="${-mount_spacing} 0 0" rpy="0 0 0" />
   </joint>
   <!-- Bring in simulation data for Gazebo. -->

Commit message: chanked link_base to base_link

File: robot/jackal/urdf/jackal.urdf.xacro (robot description, xacro)
@@ -80,8 +80,8 @@
     <origin xyz="${-wheelbase/2} ${-track/2} ${wheel_vertical_offset}" rpy="0 0 0" />
   </xacro:wheel>
-  <link name="link_base"></link>
-  <joint name="link_base_joint" type="fixed">
+  <link name="base_link"></link>
+  <joint name="base_link_joint" type="fixed">
     <origin xyz="0 0 0" rpy="0 0 0" />
-    <parent link="link_base"/>
+    <parent link="base_link"/>
     <child link="chassis_link" />
   </joint>
