Commit message: tiago

File: robot/tiago/urdf/arm/arm.urdf.xacro (robot description, xacro)
@@ -48,5 +48,5 @@
         <origin xyz="0 0 0" rpy="0 0 0" />
         <geometry>
-          <mesh filename="package://arena-simulation-setup/robot/tiago/meshes/arm/arm_1.stl" scale="1 ${-1 * tiago_dual} ${reflect}"/>
+          <mesh filename="package://arena-simulation-setup/robot/tiago/urdf/meshes/arm/arm_1.stl" scale="1 ${-1 * tiago_dual} ${reflect}"/>
         </geometry>
         <material name="White"/>
@@ -55,5 +55,5 @@
         <origin xyz="0 0 0" rpy="0 0 0" />
         <geometry>
-          <mesh filename="package://arena-simulation-setup/robot/tiago/meshes/arm/arm_1_collision.dae" scale="1 ${-1 * tiago_dual} ${reflect}"/>
+          <mesh filename="package://arena-simulation-setup/robot/tiago/urdf/meshes/arm/arm_1_collision.dae" scale="1 ${-1 * tiago_dual} ${reflect}"/>
         </geometry>
       </collision>
@@ -85,5 +85,5 @@
         <origin xyz="0 0 0" rpy="${0 * deg_to_rad} ${0 * deg_to_rad} ${0 * deg_to_rad}" />
         <geometry>
-          <mesh filename="package://arena-simulation-setup/robot/tiago/meshes/arm/arm_2.stl" scale="1 1 ${reflect}"/>
+          <mesh filename="package://arena-simulation-setup/robot/tiago/urdf/meshes/arm/arm_2.stl" scale="1 1 ${reflect}"/>
         </geometry>
         <material name="DarkGrey" />
@@ -93,5 +93,5 @@
         <origin xyz="0 0 0" rpy="${0 * deg_to_rad} ${0 * deg_to_rad} ${0 * deg_to_rad}" />
         <geometry>
-          <mesh filename="package://arena-simulation-setup/robot/tiago/meshes/arm/arm_2_collision.dae" scale="1 1 ${reflect}"/>
+          <mesh filename="package://arena-simulation-setup/robot/tiago/urdf/meshes/arm/arm_2_collision.dae" scale="1 1 ${reflect}"/>
         </geometry>
       </collision>
@@ -123,5 +123,5 @@
         <origin xyz="0 0 0" rpy="0 0 0" />
         <geometry>
-          <mesh filename="package://arena-simulation-setup/robot/tiago/meshes/arm/arm_3.stl" scale="1 1 ${reflect}"/>
+          <mesh filename="package://arena-simulation-setup/robot/tiago/urdf/meshes/arm/arm_3.stl" scale="1 1 ${reflect}"/>
         </geometry>
         <material name="DarkGrey" />
@@ -130,5 +130,5 @@
         <origin xyz="0 0 0" rpy="0 0 0" />
         <geometry>
-          <mesh filename="package://arena-simulation-setup/robot/tiago/meshes/arm/arm_3_collision.dae" scale="1 1 ${reflect}"/>
+          <mesh filename="package://arena-simulation-setup/robot/tiago/urdf/meshes/arm/arm_3_collision.dae" scale="1 1 ${reflect}"/>
         </geometry>
       </collision>
@@ -163,5 +163,5 @@
         <origin xyz="0 0 0" rpy="0 0 0" />
         <geometry>
-          <mesh filename="package://arena-simulation-setup/robot/tiago/meshes/arm/arm_4.stl" scale="${reflect} ${reflect} ${reflect}"/>
+          <mesh filename="package://arena-simulation-setup/robot/tiago/urdf/meshes/arm/arm_4.stl" scale="${reflect} ${reflect} ${reflect}"/>
         </geometry>
         <material name="DarkGrey" />
@@ -170,5 +170,5 @@
         <origin xyz="0 0 0" rpy="0 0 0" />
         <geometry>
-          <mesh filename="package://arena-simulation-setup/robot/tiago/meshes/arm/arm_4_collision.dae" scale="${reflect} ${reflect} ${reflect}"/>
+          <mesh filename="package://arena-simulation-setup/robot/tiago/urdf/meshes/arm/arm_4_collision.dae" scale="${reflect} ${reflect} ${reflect}"/>
         </geometry>
       </collision>

File: robot/tiago/urdf/arm/wrist.urdf.xacro (robot description, xacro)
@@ -49,5 +49,5 @@
         <origin xyz="0 0 0" rpy="0 0 0" />
         <geometry>
-          <mesh filename="package://arena-simulation-setup/robot/tiago/meshes/arm/arm_5-${wrist_model}.stl" scale="${reflect} ${reflect} ${reflect}"/>
+          <mesh filename="package://arena-simulation-setup/robot/tiago/urdf/meshes/arm/arm_5-${wrist_model}.stl" scale="${reflect} ${reflect} ${reflect}"/>
         </geometry>
         <material name="LightGrey" />
@@ -56,5 +56,5 @@
         <origin xyz="0 0 0" rpy="0 0 0" />
         <geometry>
-          <mesh filename="package://arena-simulation-setup/robot/tiago/meshes/arm/arm_5_collision-${wrist_model}.dae" scale="${reflect} ${reflect} ${reflect}"/>
+          <mesh filename="package://arena-simulation-setup/robot/tiago/urdf/meshes/arm/arm_5_collision-${wrist_model}.dae" scale="${reflect} ${reflect} ${reflect}"/>
         </geometry>
       </collision>
@@ -91,5 +91,5 @@
         <origin xyz="0 0 0" rpy="0 0 0" />
         <geometry>
-          <mesh filename="package://arena-simulation-setup/robot/tiago/meshes/arm/arm_6-${wrist_model}.stl" scale="${reflect} 1 1"/>
+          <mesh filename="package://arena-simulation-setup/robot/tiago/urdf/meshes/arm/arm_6-${wrist_model}.stl" scale="${reflect} 1 1"/>
         </geometry>
         <material name="LightGrey" />
@@ -98,5 +98,5 @@
         <origin xyz="0 0 0" rpy="0 0 0" />
         <geometry>
-          <mesh filename="package://arena-simulation-setup/robot/tiago/meshes/arm/arm_6_collision-${wrist_model}.dae" scale="${reflect} 1 1"/>
+          <mesh filename="package://arena-simulation-setup/robot/tiago/urdf/meshes/arm/arm_6_collision-${wrist_model}.dae" scale="${reflect} 1 1"/>
         </geometry>
       </collision>

File: robot/tiago/urdf/head/head.urdf.xacro (robot description, xacro)
@@ -41,5 +41,5 @@
         <origin xyz="0 0 0" rpy="0 0 0"/>
         <geometry>
-          <mesh filename="package://arena-simulation-setup/robot/tiago/meshes/head/head_1.stl" scale="1 1 1"/>
+          <mesh filename="package://arena-simulation-setup/robot/tiago/urdf/meshes/head/head_1.stl" scale="1 1 1"/>
         </geometry>
         <material name="White" />
@@ -48,5 +48,5 @@
         <origin xyz="0.0 0 0" rpy="0 0 0.0" />
         <geometry>
-          <mesh filename="package://arena-simulation-setup/robot/tiago/meshes/head/head_1_collision.dae" scale="1 1 1"/>
+          <mesh filename="package://arena-simulation-setup/robot/tiago/urdf/meshes/head/head_1_collision.dae" scale="1 1 1"/>
         </geometry>
         <material name="White" />
@@ -90,5 +90,5 @@
         <origin xyz="0 0 0" rpy="0 0 0" />
         <geometry>
-          <mesh filename="package://arena-simulation-setup/robot/tiago/meshes/head/head_2.stl" scale="1 1 1"/>
+          <mesh filename="package://arena-simulation-setup/robot/tiago/urdf/meshes/head/head_2.stl" scale="1 1 1"/>
         </geometry>
         <material name="White" />
@@ -97,5 +97,5 @@
         <origin xyz="0 0 0" rpy="0 0 0" />
         <geometry>
-          <mesh filename="package://arena-simulation-setup/robot/tiago/meshes/head/head_2_collision.dae" scale="1 1 1"/>
+          <mesh filename="package://arena-simulation-setup/robot/tiago/urdf/meshes/head/head_2_collision.dae" scale="1 1 1"/>
         </geometry>
       </collision>

File: robot/tiago/urdf/sensors/orbbec_astra.urdf.xacro (robot description, xacro)
@@ -37,5 +37,5 @@
         <origin xyz="0 0 0" rpy="0 0 0"/>
         <geometry>
-          <mesh filename="package://arena-simulation-setup/robot/tiago/meshes/sensors/xtion_pro_live/xtion_pro_live.dae" />
+          <mesh filename="package://arena-simulation-setup/robot/tiago/urdf/meshes/sensors/xtion_pro_live/xtion_pro_live.dae" />
         </geometry>
         <material name="Grey">

File: robot/tiago/urdf/sensors/xtion_pro_live.urdf.xacro (robot description, xacro)
@@ -36,5 +36,5 @@
         <origin xyz="0 0 0" rpy="0 0 0"/>
         <geometry>
-          <mesh filename="package://arena-simulation-setup/robot/tiago/meshes/sensors/xtion_pro_live/xtion_pro_live.dae" />
+          <mesh filename="package://arena-simulation-setup/robot/tiago/urdf/meshes/sensors/xtion_pro_live/xtion_pro_live.dae" />
         </geometry>
         <material name="Grey">

File: robot/tiago/urdf/tiago.urdf.xacro (robot description, xacro)
@@ -18,5 +18,5 @@
     <xacro:arg name="end_effector" default="false"/> <!-- false, pal-gripper, pal-hey5, schunk-wsg-->
     <xacro:arg name="ft_sensor" default="false"/> <!-- false, schunk-ft -->
-    <xacro:arg name="laser_model" default="sick-571"/> <!-- false, hokuyo, sick-551, sick-561, sick-571-->
+    <xacro:arg name="laser_model" default="sick-551"/> <!-- false, hokuyo, sick-551, sick-561, sick-571-->
     <xacro:arg name="camera_model" default="false"/> <!-- false, orbbec-astra, orbbec-astra-pro, asus-xtion -->
     <xacro:arg name="has_thermal_camera" default="false"/>
@@ -89,5 +89,5 @@
   <!-- Now we can start using the macros included above to define the actual robot -->
   <xacro:if value="${base_type == 'pmb2'}">
-    <xacro:base_sensors name="base" laser_model="$(arg laser_model)" sonars="true" microphone="true"/>
+    <xacro:base_sensors name="base" laser_model="$(arg laser_model)" sonars="true" microphone="true" />
   </xacro:if>
   <xacro:if value="${base_type == 'omni_base'}">

File: robot/tiago/urdf/torso/torso.urdf.xacro (robot description, xacro)
@@ -32,5 +32,5 @@
       <origin rpy="0 0 0" xyz="0 0 0" />
       <geometry>
-        <mesh filename="package://arena-simulation-setup/robot/tiago/meshes/torso/torso_fix.stl" scale="1 1 1"/>
+        <mesh filename="package://arena-simulation-setup/robot/tiago/urdf/meshes/torso/torso_fix.stl" scale="1 1 1"/>
       </geometry>
       <material name="LightGrey"/>
@@ -100,5 +100,5 @@
       <origin rpy="0 0 0" xyz="0 0 0" />
        <geometry>
-        <mesh filename="package://arena-simulation-setup/robot/tiago/meshes/torso/torso_lift_with_arm.stl" scale="1 1 1"/>
+        <mesh filename="package://arena-simulation-setup/robot/tiago/urdf/meshes/torso/torso_lift_with_arm.stl" scale="1 1 1"/>
       </geometry>
       <material name="White"/>
@@ -107,5 +107,5 @@
       <origin rpy="0 0 0" xyz="0 0 0" />
        <geometry>
-        <mesh filename="package://arena-simulation-setup/robot/tiago/meshes/torso/torso_lift_collision_core.dae" scale="1 1 1"/>
+        <mesh filename="package://arena-simulation-setup/robot/tiago/urdf/meshes/torso/torso_lift_collision_core.dae" scale="1 1 1"/>
       </geometry>
       <material name="LightGrey"/>
@@ -114,5 +114,5 @@
       <origin rpy="0 0 0" xyz="0 0 0" />
        <geometry>
-        <mesh filename="package://arena-simulation-setup/robot/tiago/meshes/torso/torso_lift_collision_shoulder.dae" scale="1 1 1"/>
+        <mesh filename="package://arena-simulation-setup/robot/tiago/urdf/meshes/torso/torso_lift_collision_shoulder.dae" scale="1 1 1"/>
       </geometry>
       <material name="LightGrey"/>
@@ -121,5 +121,5 @@
       <origin rpy="0 0 0" xyz="0 0 0" />
        <geometry>
-        <mesh filename="package://arena-simulation-setup/robot/tiago/meshes/torso/torso_lift_collision_neck.dae" scale="1 1 1"/>
+        <mesh filename="package://arena-simulation-setup/robot/tiago/urdf/meshes/torso/torso_lift_collision_neck.dae" scale="1 1 1"/>
       </geometry>
       <material name="LightGrey"/>
