Commit message: rto

File: robot/rto/urdf/components/rto_body.urdf.xacro (robot description, xacro)
@@ -20,5 +20,5 @@
                 <origin xyz="0.01 0 0" rpy="0 0 ${M_PI/2}"/>
                 <geometry>
-                    <mesh filename="package://arena-simulation-setup/robot/rto/meshes/parts/rto_base.dae"
+                    <mesh filename="package://arena-simulation-setup/robot/rto/urdf/meshes/parts/rto_base.dae"
                         scale="${M_SCALE} ${M_SCALE} ${M_SCALE}"/>
                 </geometry>

File: robot/rto/urdf/components/rto_parts.urdf.xacro (robot description, xacro)
@@ -19,5 +19,5 @@
                 <origin xyz="0 0 0" rpy="0 0 0"/>
                 <geometry>
-                    <mesh filename="package://arena-simulation-setup/robot/rto/meshes/parts/rto_wheel.dae" scale="${M_SCALE} ${M_SCALE} ${M_SCALE}"/>
+                    <mesh filename="package://arena-simulation-setup/robot/rto/urdf/meshes/parts/rto_wheel.dae" scale="${M_SCALE} ${M_SCALE} ${M_SCALE}"/>
                 </geometry>
             </visual>
@@ -77,5 +77,5 @@
                 <origin xyz="0 0 0" rpy="0 0 0"/>
                 <geometry>
-                    <mesh filename="package://arena-simulation-setup/robot/rto/meshes/parts/angle_bracket_usb_hub.dae" scale="${M_SCALE} ${M_SCALE} ${M_SCALE}"/>
+                    <mesh filename="package://arena-simulation-setup/robot/rto/urdf/meshes/parts/angle_bracket_usb_hub.dae" scale="${M_SCALE} ${M_SCALE} ${M_SCALE}"/>
                 </geometry>
             </visual>
@@ -153,5 +153,5 @@
                 <origin xyz="0 0 0" rpy="0 0 0"/>
                 <geometry>
-                    <mesh filename="package://arena-simulation-setup/robot/rto/meshes/parts/bracket.dae" scale="0.001 ${scale} ${scale}"/>
+                    <mesh filename="package://arena-simulation-setup/robot/rto/urdf/meshes/parts/bracket.dae" scale="0.001 ${scale} ${scale}"/>
                 </geometry>
                 <material name="dark_grey"/>

File: robot/rto/urdf/components/rto_platform.urdf (robot description, URDF)
Before this commit: robot rto, 7 links, 6 joints
Links:
- link anglebracketusb_link: geometry visual mesh filename=package://arena-simulation-setup/robot/rto/urdf/meshes/part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 scale=0.01 0.01 0.01
- link base_link: geometry collision cylinder length=0.05 radius=0.18; visual mesh filename=package://arena-simulation-setup/robot/rto/urdf/meshes/part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 scale=0.01 0.01 0.01
- link wheel0_link: geometry visual mesh filename=package://arena-simulation-setup/robot/rto/urdf/meshes/part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 scale=0.01 0.01 0.01
- link wheel1_link: geometry visual mesh filename=package://arena-simulation-setup/robot/rto/urdf/meshes/part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 scale=0.01 0.01 0.01
- link wheel2_link: geometry visual mesh filename=package://arena-simulation-setup/robot/rto/urdf/meshes/part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 scale=0.01 0.01 0.01

File: robot/rto/urdf/components/rto_platform_kinect.urdf (robot description, URDF)
Before this commit: robot rto, 8 links, 7 joints
Links:
- link anglebracketusb_link: geometry visual mesh filename=package://arena-simulation-setup/robot/rto/urdf/meshes/part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 scale=0.01 0.01 0.01
- link base_link: geometry collision cylinder length=0.05 radius=0.18; visual mesh filename=package://arena-simulation-setup/robot/rto/urdf/meshes/part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 scale=0.01 0.01 0.01
- link kinect_link: geometry collision box size=0.064 0.121 0.0381; visual mesh filename=package://arena-simulation-setup/robot/rto/urdf/meshes/sens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
- link wheel0_link: geometry visual mesh filename=package://arena-simulation-setup/robot/rto/urdf/meshes/part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 scale=0.01 0.01 0.01
- link wheel1_link: geometry visual mesh filename=package://arena-simulation-setup/robot/rto/urdf/meshes/part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 scale=0.01 0.01 0.01
- link wheel2_link: geometry visual mesh filename=package://arena-simulation-setup/robot/rto/urdf/meshes/part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 scale=0.01 0.01 0.01

File: robot/rto/urdf/realsense2/urdf/_d415.urdf.xacro (robot description, xacro)
@@ -3,36 +3,30 @@
 License: Apache 2.0. See LICENSE file in root directory.
 Copyright(c) 2017 Intel Corporation. All Rights Reserved
-This is the URDF model for the Intel RealSense 430 camera, in its
+This is the URDF model for the Intel RealSense 415 camera, in its
 aluminum peripherial evaluation case.
 -->
-<robot name="sensor_d435" xmlns:xacro="http://ros.org/wiki/xacro">
+<robot name="sensor_d415" xmlns:xacro="http://ros.org/wiki/xacro">
   <!-- Includes -->
-  <xacro:include filename="$(find arena-simulation-setup)/robot/rto/realsense2/urdf/_materials.urdf.xacro" />
-  <xacro:include filename="$(find arena-simulation-setup)/robot/rto/realsense2/urdf/_usb_plug.urdf.xacro" />
-  <xacro:macro name="sensor_d435" params="parent *origin name:=camera use_nominal_extrinsics:=false add_plug:=false use_mesh:=true">
+  <xacro:include filename="$(find arena-simulation-setup)/robot/rto/urdf/realsense2/urdf/_materials.urdf.xacro" />
+  <xacro:include filename="$(find arena-simulation-setup)/robot/rto/urdf/realsense2/urdf/_usb_plug.urdf.xacro" />
+  <xacro:macro name="sensor_d415" params="parent *origin  name:=camera  use_nominal_extrinsics:=false add_plug:=false use_mesh:=true">
     <xacro:property name="M_PI" value="3.1415926535897931" />
     <!-- The following values are approximate, and the camera node
      publishing TF values with actual calibrated camera extrinsic values -->
-    <xacro:property name="d435_cam_depth_to_infra1_offset" value="0.0"/>
-    <xacro:property name="d435_cam_depth_to_infra2_offset" value="-0.050"/>
-    <xacro:property name="d435_cam_depth_to_color_offset" value="0.015"/>
+    <xacro:property name="d415_cam_depth_to_infra1_offset" value="0.0"/>
+    <xacro:property name="d415_cam_depth_to_infra2_offset" value="-0.055"/>
+    <xacro:property name="d415_cam_depth_to_color_offset" value="0.015"/>
     <!-- The following values model the aluminum peripherial case for the
-  	D435 camera, with the camera joint represented by the actual
+  	d415 camera, with the camera joint represented by the actual
   	peripherial camera tripod mount -->
-    <xacro:property name="d435_cam_width" value="0.090"/>
-    <xacro:property name="d435_cam_height" value="0.025"/>
-    <xacro:property name="d435_cam_depth" value="0.02505"/>
-    <xacro:property name="d435_cam_mount_from_center_offset" value="0.0149"/>
-    <!-- glass cover is 0.1 mm inwards from front aluminium plate -->
-    <xacro:property name="d435_glass_to_front" value="0.1e-3"/>
-    <!-- see datasheet Revision 007, Fig. 4-4 page 65 -->
-    <xacro:property name="d435_zero_depth_to_glass" value="4.2e-3"/>
-    <!-- convenience precomputation to avoid clutter-->
-    <xacro:property name="d435_mesh_x_offset" value="${d435_cam_mount_from_center_offset-d435_glass_to_front-d435_zero_depth_to_glass}"/>
-    <!-- The following offset is relative the the physical D435 camera peripherial
+    <xacro:property name="d415_cam_width" value="0.099"/>
+    <xacro:property name="d415_cam_height" value="0.023"/>
+    <xacro:property name="d415_cam_depth" value="0.02005"/>
+    <xacro:property name="d415_cam_mount_from_center_offset" value="0.00987"/>
+    <!-- The following offset is relative the the physical d415 camera peripherial
   	camera tripod mount -->
-    <xacro:property name="d435_cam_depth_px" value="${d435_cam_mount_from_center_offset}"/>
-    <xacro:property name="d435_cam_depth_py" value="0.0175"/>
-    <xacro:property name="d435_cam_depth_pz" value="${d435_cam_height/2}"/>
+    <xacro:property name="d415_cam_depth_px" value="${d415_cam_mount_from_center_offset}"/>
+    <xacro:property name="d415_cam_depth_py" value="0.020"/>
+    <xacro:property name="d415_cam_depth_pz" value="${d415_cam_height/2}"/>
     <!-- camera body, with origin at bottom screw mount -->
     <joint name="${name}_joint" type="fixed">
@@ -43,5 +37,5 @@
     <link name="${name}_bottom_screw_frame"/>
     <joint name="${name}_link_joint" type="fixed">
-      <origin xyz="${d435_mesh_x_offset} ${d435_cam_depth_py} ${d435_cam_depth_pz}" rpy="0 0 0"/>
+      <origin xyz="0 ${d415_cam_depth_py} ${d415_cam_depth_pz}" rpy="0 0 0"/>
       <parent link="${name}_bottom_screw_frame"/>
       <child link="${name}_link" />
@@ -50,27 +44,26 @@
       <visual>
         <xacro:if value="${use_mesh}">
-          <!-- the mesh origin is at front plate in between the two infrared camera axes -->
-          <origin xyz="${d435_zero_depth_to_glass + d435_glass_to_front} ${-d435_cam_depth_py} 0" rpy="${M_PI/2} 0 ${M_PI/2}"/>
+          <origin xyz="${d415_cam_mount_from_center_offset} ${-d415_cam_depth_py} 0" rpy="${M_PI/2} 0 ${M_PI/2}"/>
           <geometry>
-            <mesh filename="package://package://arena-simulation-setup/robot/rto/realsense2/meshes/meshes/d435.dae" />
+            <mesh filename="package://package://arena-simulation-setup/robot/rto/urdf/realsense2/urdf/meshes/urdf/meshes/d415.stl" />
           </geometry>
+          <material name="aluminum"/>
         </xacro:if>
         <xacro:unless value="${use_mesh}">
-          <origin xyz="0 ${-d435_cam_depth_py} 0" rpy="0 0 0"/>
+          <origin xyz="0 ${-d415_cam_depth_py} 0" rpy="0 0 0"/>
           <geometry>
-            <box size="${d435_cam_depth} ${d435_cam_width} ${d435_cam_height}"/>
+            <box size="${d415_cam_depth} ${d415_cam_width} ${d415_cam_height}"/>
           </geometry>
-          <material name="aluminum"/>
         </xacro:unless>
       </visual>
       <collision>
-        <origin xyz="0 ${-d435_cam_depth_py} 0" rpy="0 0 0"/>
+        <origin xyz="0 ${-d415_cam_depth_py} 0" rpy="0 0 0"/>
         <geometry>
-          <box size="${d435_cam_depth} ${d435_cam_width} ${d435_cam_height}"/>
+        <box size="${d415_cam_depth} ${d415_cam_width} ${d415_cam_height}"/>
         </geometry>
       </collision>
       <inertial>
+        <mass value="0.072" />
         <!-- The following are not reliable values, and should not be used for modeling -->
-        <mass value="0.072" />
         <origin xyz="0 0 0" />
         <inertia ixx="0.003881243" ixy="0.0" ixz="0.0" iyy="0.000498940" iyz="0.0" izz="0.003879257" />
@@ -94,5 +87,5 @@
       <!-- camera left IR joints and links -->
       <joint name="${name}_infra1_joint" type="fixed">
-        <origin xyz="0 ${d435_cam_depth_to_infra1_offset} 0" rpy="0 0 0" />
+        <origin xyz="0 ${d415_cam_depth_to_infra1_offset} 0" rpy="0 0 0" />
         <parent link="${name}_link" />
         <child link="${name}_infra1_frame" />
@@ -107,5 +100,5 @@
       <!-- camera right IR joints and links -->
       <joint name="${name}_infra2_joint" type="fixed">
-        <origin xyz="0 ${d435_cam_depth_to_infra2_offset} 0" rpy="0 0 0" />
+        <origin xyz="0 ${d415_cam_depth_to_infra2_offset} 0" rpy="0 0 0" />
         <parent link="${name}_link" />
         <child link="${name}_infra2_frame" />
@@ -120,5 +113,5 @@
       <!-- camera color joints and links -->
       <joint name="${name}_color_joint" type="fixed">
-        <origin xyz="0 ${d435_cam_depth_to_color_offset} 0" rpy="0 0 0" />
+        <origin xyz="0 ${d415_cam_depth_to_color_offset} 0" rpy="0 0 0" />
         <parent link="${name}_link" />
         <child link="${name}_color_frame" />
@@ -134,5 +127,5 @@
     <xacro:if value="${add_plug}">
       <xacro:usb_plug parent="${name}_link" name="${name}_usb_plug">
-        <origin xyz="${d435_cam_mount_from_center_offset - 0.02095} ${-d435_cam_depth_py - 0.0353} 0" rpy="0 0 0"/>
+        <origin xyz="${d415_cam_mount_from_center_offset - 0.01587} ${-d415_cam_depth_py - 0.0358} 0" rpy="0 0 0"/>
       </xacro:usb_plug>
     </xacro:if>

File: robot/rto/urdf/realsense2/urdf/_d435.urdf.xacro (robot description, xacro)
@@ -3,30 +3,36 @@
 License: Apache 2.0. See LICENSE file in root directory.
 Copyright(c) 2017 Intel Corporation. All Rights Reserved
-This is the URDF model for the Intel RealSense 415 camera, in its
+This is the URDF model for the Intel RealSense 430 camera, in its
 aluminum peripherial evaluation case.
 -->
-<robot name="sensor_d415" xmlns:xacro="http://ros.org/wiki/xacro">
+<robot name="sensor_d435" xmlns:xacro="http://ros.org/wiki/xacro">
   <!-- Includes -->
-  <xacro:include filename="$(find arena-simulation-setup)/robot/rto/realsense2/urdf/_materials.urdf.xacro" />
-  <xacro:include filename="$(find arena-simulation-setup)/robot/rto/realsense2/urdf/_usb_plug.urdf.xacro" />
-  <xacro:macro name="sensor_d415" params="parent *origin  name:=camera  use_nominal_extrinsics:=false add_plug:=false use_mesh:=true">
+  <xacro:include filename="$(find arena-simulation-setup)/robot/rto/urdf/realsense2/urdf/_materials.urdf.xacro" />
+  <xacro:include filename="$(find arena-simulation-setup)/robot/rto/urdf/realsense2/urdf/_usb_plug.urdf.xacro" />
+  <xacro:macro name="sensor_d435" params="parent *origin name:=camera use_nominal_extrinsics:=false add_plug:=false use_mesh:=true">
     <xacro:property name="M_PI" value="3.1415926535897931" />
     <!-- The following values are approximate, and the camera node
      publishing TF values with actual calibrated camera extrinsic values -->
-    <xacro:property name="d415_cam_depth_to_infra1_offset" value="0.0"/>
-    <xacro:property name="d415_cam_depth_to_infra2_offset" value="-0.055"/>
-    <xacro:property name="d415_cam_depth_to_color_offset" value="0.015"/>
+    <xacro:property name="d435_cam_depth_to_infra1_offset" value="0.0"/>
+    <xacro:property name="d435_cam_depth_to_infra2_offset" value="-0.050"/>
+    <xacro:property name="d435_cam_depth_to_color_offset" value="0.015"/>
     <!-- The following values model the aluminum peripherial case for the
-  	d415 camera, with the camera joint represented by the actual
+  	D435 camera, with the camera joint represented by the actual
   	peripherial camera tripod mount -->
-    <xacro:property name="d415_cam_width" value="0.099"/>
-    <xacro:property name="d415_cam_height" value="0.023"/>
-    <xacro:property name="d415_cam_depth" value="0.02005"/>
-    <xacro:property name="d415_cam_mount_from_center_offset" value="0.00987"/>
-    <!-- The following offset is relative the the physical d415 camera peripherial
+    <xacro:property name="d435_cam_width" value="0.090"/>
+    <xacro:property name="d435_cam_height" value="0.025"/>
+    <xacro:property name="d435_cam_depth" value="0.02505"/>
+    <xacro:property name="d435_cam_mount_from_center_offset" value="0.0149"/>
+    <!-- glass cover is 0.1 mm inwards from front aluminium plate -->
+    <xacro:property name="d435_glass_to_front" value="0.1e-3"/>
+    <!-- see datasheet Revision 007, Fig. 4-4 page 65 -->
+    <xacro:property name="d435_zero_depth_to_glass" value="4.2e-3"/>
+    <!-- convenience precomputation to avoid clutter-->
+    <xacro:property name="d435_mesh_x_offset" value="${d435_cam_mount_from_center_offset-d435_glass_to_front-d435_zero_depth_to_glass}"/>
+    <!-- The following offset is relative the the physical D435 camera peripherial
   	camera tripod mount -->
-    <xacro:property name="d415_cam_depth_px" value="${d415_cam_mount_from_center_offset}"/>
-    <xacro:property name="d415_cam_depth_py" value="0.020"/>
-    <xacro:property name="d415_cam_depth_pz" value="${d415_cam_height/2}"/>
+    <xacro:property name="d435_cam_depth_px" value="${d435_cam_mount_from_center_offset}"/>
+    <xacro:property name="d435_cam_depth_py" value="0.0175"/>
+    <xacro:property name="d435_cam_depth_pz" value="${d435_cam_height/2}"/>
     <!-- camera body, with origin at bottom screw mount -->
     <joint name="${name}_joint" type="fixed">
@@ -37,5 +43,5 @@
     <link name="${name}_bottom_screw_frame"/>
     <joint name="${name}_link_joint" type="fixed">
-      <origin xyz="0 ${d415_cam_depth_py} ${d415_cam_depth_pz}" rpy="0 0 0"/>
+      <origin xyz="${d435_mesh_x_offset} ${d435_cam_depth_py} ${d435_cam_depth_pz}" rpy="0 0 0"/>
       <parent link="${name}_bottom_screw_frame"/>
       <child link="${name}_link" />
@@ -44,26 +50,27 @@
       <visual>
         <xacro:if value="${use_mesh}">
-          <origin xyz="${d415_cam_mount_from_center_offset} ${-d415_cam_depth_py} 0" rpy="${M_PI/2} 0 ${M_PI/2}"/>
+          <!-- the mesh origin is at front plate in between the two infrared camera axes -->
+          <origin xyz="${d435_zero_depth_to_glass + d435_glass_to_front} ${-d435_cam_depth_py} 0" rpy="${M_PI/2} 0 ${M_PI/2}"/>
           <geometry>
-            <mesh filename="package://package://arena-simulation-setup/robot/rto/realsense2/meshes/meshes/d415.stl" />
+            <mesh filename="package://package://arena-simulation-setup/robot/rto/urdf/realsense2/urdf/meshes/urdf/meshes/d435.dae" />
+          </geometry>
+        </xacro:if>
+        <xacro:unless value="${use_mesh}">
+          <origin xyz="0 ${-d435_cam_depth_py} 0" rpy="0 0 0"/>
+          <geometry>
+            <box size="${d435_cam_depth} ${d435_cam_width} ${d435_cam_height}"/>
           </geometry>
           <material name="aluminum"/>
-        </xacro:if>
-        <xacro:unless value="${use_mesh}">
-          <origin xyz="0 ${-d415_cam_depth_py} 0" rpy="0 0 0"/>
-          <geometry>
-            <box size="${d415_cam_depth} ${d415_cam_width} ${d415_cam_height}"/>
-          </geometry>
         </xacro:unless>
       </visual>
       <collision>
-        <origin xyz="0 ${-d415_cam_depth_py} 0" rpy="0 0 0"/>
+        <origin xyz="0 ${-d435_cam_depth_py} 0" rpy="0 0 0"/>
         <geometry>
-        <box size="${d415_cam_depth} ${d415_cam_width} ${d415_cam_height}"/>
+          <box size="${d435_cam_depth} ${d435_cam_width} ${d435_cam_height}"/>
         </geometry>
       </collision>
       <inertial>
+        <!-- The following are not reliable values, and should not be used for modeling -->
         <mass value="0.072" />
-        <!-- The following are not reliable values, and should not be used for modeling -->
         <origin xyz="0 0 0" />
         <inertia ixx="0.003881243" ixy="0.0" ixz="0.0" iyy="0.000498940" iyz="0.0" izz="0.003879257" />
@@ -87,5 +94,5 @@
       <!-- camera left IR joints and links -->
       <joint name="${name}_infra1_joint" type="fixed">
-        <origin xyz="0 ${d415_cam_depth_to_infra1_offset} 0" rpy="0 0 0" />
+        <origin xyz="0 ${d435_cam_depth_to_infra1_offset} 0" rpy="0 0 0" />
         <parent link="${name}_link" />
         <child link="${name}_infra1_frame" />
@@ -100,5 +107,5 @@
       <!-- camera right IR joints and links -->
       <joint name="${name}_infra2_joint" type="fixed">
-        <origin xyz="0 ${d415_cam_depth_to_infra2_offset} 0" rpy="0 0 0" />
+        <origin xyz="0 ${d435_cam_depth_to_infra2_offset} 0" rpy="0 0 0" />
         <parent link="${name}_link" />
         <child link="${name}_infra2_frame" />
@@ -113,5 +120,5 @@
       <!-- camera color joints and links -->
       <joint name="${name}_color_joint" type="fixed">
-        <origin xyz="0 ${d415_cam_depth_to_color_offset} 0" rpy="0 0 0" />
+        <origin xyz="0 ${d435_cam_depth_to_color_offset} 0" rpy="0 0 0" />
         <parent link="${name}_link" />
         <child link="${name}_color_frame" />
@@ -127,5 +134,5 @@
     <xacro:if value="${add_plug}">
       <xacro:usb_plug parent="${name}_link" name="${name}_usb_plug">
-        <origin xyz="${d415_cam_mount_from_center_offset - 0.01587} ${-d415_cam_depth_py - 0.0358} 0" rpy="0 0 0"/>
+        <origin xyz="${d435_cam_mount_from_center_offset - 0.02095} ${-d435_cam_depth_py - 0.0353} 0" rpy="0 0 0"/>
       </xacro:usb_plug>
     </xacro:if>

File: robot/rto/urdf/realsense2/urdf/_d435i.urdf.xacro (robot description, xacro)
@@ -7,6 +7,6 @@
 -->
 <robot name="sensor_d435i" xmlns:xacro="http://ros.org/wiki/xacro">
-  <xacro:include filename="$(find arena-simulation-setup)/robot/rto/realsense2/urdf/_d435.urdf.xacro"/>
-  <xacro:include filename="$(find arena-simulation-setup)/robot/rto/realsense2/urdf/_d435i_imu_modules.urdf.xacro"/>
+  <xacro:include filename="$(find arena-simulation-setup)/robot/rto/urdf/realsense2/urdf/_d435.urdf.xacro"/>
+  <xacro:include filename="$(find arena-simulation-setup)/robot/rto/urdf/realsense2/urdf/_d435i_imu_modules.urdf.xacro"/>
   <xacro:macro name="sensor_d435i" params="parent *origin name:=camera use_nominal_extrinsics:=false">
     <xacro:sensor_d435 parent="${parent}" name="${name}" use_nominal_extrinsics="${use_nominal_extrinsics}">

File: robot/rto/urdf/realsense2/urdf/_d455.urdf.xacro (robot description, xacro)
@@ -8,6 +8,6 @@
 <robot name="sensor_d455" xmlns:xacro="http://ros.org/wiki/xacro">
   <!-- Includes -->
-  <xacro:include filename="$(find arena-simulation-setup)/robot/rto/realsense2/urdf/_materials.urdf.xacro" />
-  <xacro:include filename="$(find arena-simulation-setup)/robot/rto/realsense2/urdf/_usb_plug.urdf.xacro" />
+  <xacro:include filename="$(find arena-simulation-setup)/robot/rto/urdf/realsense2/urdf/_materials.urdf.xacro" />
+  <xacro:include filename="$(find arena-simulation-setup)/robot/rto/urdf/realsense2/urdf/_usb_plug.urdf.xacro" />
   <xacro:macro name="sensor_d455" params="parent *origin name:=camera use_nominal_extrinsics:=false">
     <xacro:arg name="add_plug" default="false" />
@@ -55,5 +55,5 @@
         <geometry>
           <!-- <box size="${d455_cam_depth} ${d455_cam_width} ${d455_cam_height}"/> -->
-	        <mesh filename="package://package://arena-simulation-setup/robot/rto/realsense2/meshes/meshes/d455.stl" scale="0.001 0.001 0.001" />
+	        <mesh filename="package://package://arena-simulation-setup/robot/rto/urdf/realsense2/urdf/meshes/urdf/meshes/d455.stl" scale="0.001 0.001 0.001" />
         </geometry>
         <material name="aluminum"/>

File: robot/rto/urdf/realsense2/urdf/_l515.urdf.xacro (robot description, xacro)
@@ -8,6 +8,6 @@
 <robot name="sensor_l515" xmlns:xacro="http://ros.org/wiki/xacro">
   <!-- Includes -->
-  <xacro:include filename="$(find arena-simulation-setup)/robot/rto/realsense2/urdf/_materials.urdf.xacro" />
-  <xacro:include filename="$(find arena-simulation-setup)/robot/rto/realsense2/urdf/_usb_plug.urdf.xacro" /> <!-- this specific plug does not apply to L515 -->
+  <xacro:include filename="$(find arena-simulation-setup)/robot/rto/urdf/realsense2/urdf/_materials.urdf.xacro" />
+  <xacro:include filename="$(find arena-simulation-setup)/robot/rto/urdf/realsense2/urdf/_usb_plug.urdf.xacro" /> <!-- this specific plug does not apply to L515 -->
   <xacro:macro name="sensor_l515" params="parent *origin name:=camera use_nominal_extrinsics:=false add_plug:=false use_mesh:=true">
     <xacro:property name="M_PI" value="3.1415926535897931" />
@@ -63,5 +63,5 @@
           <origin xyz="${l515_zero_depth_to_glass} 0 ${-l515_cam_center_to_depth_pz}" rpy="${M_PI/2} 0 ${M_PI/2}"/>
           <geometry>
-              <mesh filename="package://package://arena-simulation-setup/robot/rto/realsense2/meshes/meshes/l515.dae" />
+              <mesh filename="package://package://arena-simulation-setup/robot/rto/urdf/realsense2/urdf/meshes/urdf/meshes/l515.dae" />
           </geometry>
         </xacro:if>
