Commit message: rto

File: robot/rto/urdf/realsense2/urdf/_r410.urdf.xacro (robot description, xacro)
@@ -8,5 +8,5 @@
 <robot name="sensor_r410" xmlns:xacro="http://ros.org/wiki/xacro">
   <!-- Includes -->
-  <xacro:include filename="$(find arena-simulation-setup)/robot/rto/realsense2/urdf/_materials.urdf.xacro" />
+  <xacro:include filename="$(find arena-simulation-setup)/robot/rto/urdf/realsense2/urdf/_materials.urdf.xacro" />
   <xacro:macro name="sensor_r410" params="parent *origin  name:=camera  use_nominal_extrinsics:=false">
     <xacro:property name="M_PI" value="3.1415926535897931" />
@@ -38,5 +38,5 @@
         <geometry>
           <box size="${r410_cam_width} ${r410_cam_height} ${r410_cam_depth}"/>
-          <!--<mesh filename="package://package://arena-simulation-setup/robot/rto/realsense2/meshes/meshes/r410/r410.dae" />-->
+          <!--<mesh filename="package://package://arena-simulation-setup/robot/rto/urdf/realsense2/urdf/meshes/urdf/meshes/r410/r410.dae" />-->
         </geometry>
         <material name="aluminum"/>

File: robot/rto/urdf/realsense2/urdf/_r430.urdf.xacro (robot description, xacro)
@@ -8,5 +8,5 @@
 <robot name="sensor_r430" xmlns:xacro="http://ros.org/wiki/xacro">
   <!-- Includes -->
-  <xacro:include filename="$(find arena-simulation-setup)/robot/rto/realsense2/urdf/_materials.urdf.xacro" />
+  <xacro:include filename="$(find arena-simulation-setup)/robot/rto/urdf/realsense2/urdf/_materials.urdf.xacro" />
   <xacro:macro name="sensor_r430" params="parent *origin name:=camera use_nominal_extrinsics:=false">
   <xacro:property name="M_PI" value="3.1415926535897931" />
@@ -39,5 +39,5 @@
         <geometry>
           <box size="${r430_cam_width} ${r430_cam_height} ${r430_cam_depth}"/>
-          <!--<mesh filename="package://package://arena-simulation-setup/robot/rto/realsense2/meshes/meshes/r430/r430.dae" />-->
+          <!--<mesh filename="package://package://arena-simulation-setup/robot/rto/urdf/realsense2/urdf/meshes/urdf/meshes/r430/r430.dae" />-->
         </geometry>
         <material name="aluminum"/>

File: robot/rto/urdf/realsense2/urdf/_usb_plug.urdf.xacro (robot description, xacro)
@@ -20,5 +20,5 @@
         <geometry>
           <!--box size="0.044850 0.008 0.0185" /-->
-          <mesh filename="package://package://arena-simulation-setup/robot/rto/realsense2/meshes/meshes/plug.stl" />
+          <mesh filename="package://package://arena-simulation-setup/robot/rto/urdf/realsense2/urdf/meshes/urdf/meshes/plug.stl" />
         </geometry>
         <material name="plastic"/>
@@ -28,5 +28,5 @@
         <geometry>
           <!--box size="0.044850 0.008 0.0185" /-->
-          <mesh filename="package://package://arena-simulation-setup/robot/rto/realsense2/meshes/meshes/plug_collision.stl" />
+          <mesh filename="package://package://arena-simulation-setup/robot/rto/urdf/realsense2/urdf/meshes/urdf/meshes/plug_collision.stl" />
         </geometry>
       </collision>

File: robot/rto/urdf/realsense2/urdf/test_d415_camera.urdf.xacro (robot description, xacro)
@@ -1,8 +1,8 @@
 <?xml version="1.0"?>
-<robot name="realsense2_camera" xmlns:xacro="http://ros.org/wiki/xacro">
+<robot name="urdf/realsense2_camera" xmlns:xacro="http://ros.org/wiki/xacro">
   <xacro:arg name="use_nominal_extrinsics" default="false" />
   <xacro:arg name="add_plug" default="false" />
   <xacro:arg name="use_mesh" default="true" />
-  <xacro:include filename="$(find arena-simulation-setup)/robot/rto/realsense2/urdf/_d415.urdf.xacro" />
+  <xacro:include filename="$(find arena-simulation-setup)/robot/rto/urdf/realsense2/urdf/_d415.urdf.xacro" />
   <link name="base_link" />
   <xacro:sensor_d415 parent="base_link" use_nominal_extrinsics="$(arg use_nominal_extrinsics)" add_plug="$(arg add_plug)" use_mesh="$(arg use_mesh)">

File: robot/rto/urdf/realsense2/urdf/test_d435_camera.urdf.xacro (robot description, xacro)
@@ -1,8 +1,8 @@
 <?xml version="1.0"?>
-<robot name="realsense2_camera" xmlns:xacro="http://ros.org/wiki/xacro">
+<robot name="urdf/realsense2_camera" xmlns:xacro="http://ros.org/wiki/xacro">
   <xacro:arg name="use_nominal_extrinsics" default="false"/>
   <xacro:arg name="add_plug" default="false" />
   <xacro:arg name="use_mesh" default="true" />
-  <xacro:include filename="$(find arena-simulation-setup)/robot/rto/realsense2/urdf/_d435.urdf.xacro" />
+  <xacro:include filename="$(find arena-simulation-setup)/robot/rto/urdf/realsense2/urdf/_d435.urdf.xacro" />
   <link name="base_link" />
   <xacro:sensor_d435 parent="base_link" use_nominal_extrinsics="$(arg use_nominal_extrinsics)" add_plug="$(arg add_plug)" use_mesh="$(arg use_mesh)">

File: robot/rto/urdf/realsense2/urdf/test_d435_multiple_cameras.urdf.xacro (robot description, xacro)
@@ -1,6 +1,6 @@
 <?xml version="1.0"?>
-<robot name="realsense2_camera" xmlns:xacro="http://ros.org/wiki/xacro">
+<robot name="urdf/realsense2_camera" xmlns:xacro="http://ros.org/wiki/xacro">
   <xacro:arg name="use_nominal_extrinsics" default="false"/>
-  <xacro:include filename="$(find arena-simulation-setup)/robot/rto/realsense2/urdf/_d435.urdf.xacro" />
+  <xacro:include filename="$(find arena-simulation-setup)/robot/rto/urdf/realsense2/urdf/_d435.urdf.xacro" />
   <link name="base_link" />
   <xacro:sensor_d435 parent="base_link" name="camera1" use_nominal_extrinsics="$(arg use_nominal_extrinsics)">

File: robot/rto/urdf/realsense2/urdf/test_d435i_camera.urdf.xacro (robot description, xacro)
@@ -1,6 +1,6 @@
 <?xml version="1.0" ?>
-<robot name="realsense2_camera" xmlns:xacro="http://www.ros.org/wiki/xacro">
+<robot name="urdf/realsense2_camera" xmlns:xacro="http://www.ros.org/wiki/xacro">
   <xacro:arg name="use_nominal_extrinsics" default="false" />
-  <xacro:include filename="$(find arena-simulation-setup)/robot/rto/realsense2/urdf/_d435i.urdf.xacro"/>
+  <xacro:include filename="$(find arena-simulation-setup)/robot/rto/urdf/realsense2/urdf/_d435i.urdf.xacro"/>
   <link name="base_link" />
   <xacro:sensor_d435i parent="base_link" use_nominal_extrinsics="$(arg use_nominal_extrinsics)">

File: robot/rto/urdf/realsense2/urdf/test_d455_camera.urdf.xacro (robot description, xacro)
@@ -1,6 +1,6 @@
 <?xml version="1.0"?>
-<robot name="realsense2_camera" xmlns:xacro="http://ros.org/wiki/xacro">
+<robot name="urdf/realsense2_camera" xmlns:xacro="http://ros.org/wiki/xacro">
   <xacro:arg name="use_nominal_extrinsics" default="false"/>
-  <xacro:include filename="$(find arena-simulation-setup)/robot/rto/realsense2/urdf/_d455.urdf.xacro" />
+  <xacro:include filename="$(find arena-simulation-setup)/robot/rto/urdf/realsense2/urdf/_d455.urdf.xacro" />
   <link name="base_link" />
   <xacro:sensor_d455 parent="base_link" use_nominal_extrinsics="$(arg use_nominal_extrinsics)">

File: robot/rto/urdf/realsense2/urdf/test_l515_camera.urdf.xacro (robot description, xacro)
@@ -1,8 +1,8 @@
 <?xml version="1.0"?>
-<robot name="realsense2_camera" xmlns:xacro="http://ros.org/wiki/xacro">
+<robot name="urdf/realsense2_camera" xmlns:xacro="http://ros.org/wiki/xacro">
   <xacro:arg name="use_nominal_extrinsics" default="false"/>
   <xacro:arg name="add_plug" default="false" />
   <xacro:arg name="use_mesh" default="true" />
-  <xacro:include filename="$(find arena-simulation-setup)/robot/rto/realsense2/urdf/_l515.urdf.xacro" />
+  <xacro:include filename="$(find arena-simulation-setup)/robot/rto/urdf/realsense2/urdf/_l515.urdf.xacro" />
   <link name="base_link" />
   <xacro:sensor_l515 parent="base_link" use_nominal_extrinsics="$(arg use_nominal_extrinsics)" add_plug="$(arg add_plug)" use_mesh="$(arg use_mesh)">

File: robot/rto/urdf/realsense2/urdf/test_r410_camera.urdf.xacro (robot description, xacro)
@@ -1,6 +1,6 @@
 <?xml version="1.0"?>
-<robot name="realsense2_camera" xmlns:xacro="http://ros.org/wiki/xacro">
+<robot name="urdf/realsense2_camera" xmlns:xacro="http://ros.org/wiki/xacro">
   <xacro:arg name="use_nominal_extrinsics" default="false"/>
-  <xacro:include filename="$(find arena-simulation-setup)/robot/rto/realsense2/urdf/_r410.urdf.xacro" />
+  <xacro:include filename="$(find arena-simulation-setup)/robot/rto/urdf/realsense2/urdf/_r410.urdf.xacro" />
   <link name="base_link" />
   <xacro:sensor_r410 parent="base_link" use_nominal_extrinsics="$(arg use_nominal_extrinsics)">

File: robot/rto/urdf/realsense2/urdf/test_r430_camera.urdf.xacro (robot description, xacro)
@@ -1,6 +1,6 @@
 <?xml version="1.0"?>
-<robot name="realsense2_camera" xmlns:xacro="http://ros.org/wiki/xacro">
+<robot name="urdf/realsense2_camera" xmlns:xacro="http://ros.org/wiki/xacro">
   <xacro:arg name="use_nominal_extrinsics" default="false"/>
-  <xacro:include filename="$(find arena-simulation-setup)/robot/rto/realsense2/urdf/_r430.urdf.xacro" />
+  <xacro:include filename="$(find arena-simulation-setup)/robot/rto/urdf/realsense2/urdf/_r430.urdf.xacro" />
   <link name="base_link" />
   <xacro:sensor_r430 parent="base_link" use_nominal_extrinsics="$(arg use_nominal_extrinsics)">
