Commit message: replaced laikago_description and added costmap

File: robot/laikago/urdf/laikago.urdf.xacro (robot description, xacro)
@@ -2,8 +2,8 @@
 <robot name="laikago" xmlns:xacro="http://www.ros.org/wiki/xacro">
     <xacro:arg name="DEBUG" default="false"/>
-    <xacro:include filename="$(find laikago_description)/xacro/const.xacro"/>
-    <xacro:include filename="$(find laikago_description)/xacro/materials.xacro"/>
-    <xacro:include filename="$(find laikago_description)/xacro/leg.xacro"/>
-    <xacro:include filename="$(find laikago_description)/xacro/gazebo.xacro"/>
+    <xacro:include filename="$(find arena-simulation-setup)/robot/laikago/xacro/const.xacro"/>
+    <xacro:include filename="$(find arena-simulation-setup)/robot/laikago/xacro/materials.xacro"/>
+    <xacro:include filename="$(find arena-simulation-setup)/robot/laikago/xacro/leg.xacro"/>
+    <xacro:include filename="$(find arena-simulation-setup)/robot/laikago/xacro/gazebo.xacro"/>
     <!-- Rollover Protection mode will add an additional stick on the top, use "true" or "false" to switch it. -->
     <xacro:property name="rolloverProtection" value="false"/>
@@ -34,5 +34,5 @@
             <origin rpy="0 0 0" xyz="0 0 0"/>
             <geometry>
-                <mesh filename="package://laikago_description/meshes/trunk.dae" scale="1 1 1"/>
+                <mesh filename="package://arena-simulation-setup/robot/laikago/meshes/trunk.dae" scale="1 1 1"/>
             </geometry>
             <material name="orange"/>

File: robot/laikago/urdf/leg.xacro (robot description, xacro)
@@ -1,5 +1,5 @@
 <?xml version="1.0"?>
 <robot xmlns:xacro="http://www.ros.org/wiki/xacro">
-    <xacro:include filename="$(find laikago_description)/xacro/transmission.xacro"/>
+    <xacro:include filename="$(find arena-simulation-setup)/robot/laikago/xacro/transmission.xacro"/>
     <xacro:macro name="leg" params="name mirror mirror_dae front_hind front_hind_dae *origin">
         <joint name="${name}_hip_joint" type="revolute">
@@ -31,5 +31,5 @@
                 </xacro:if>
                 <geometry>
-                    <mesh filename="package://laikago_description/meshes/hip.dae" scale="1 1 1"/>
+                    <mesh filename="package://arena-simulation-setup/robot/laikago/meshes/hip.dae" scale="1 1 1"/>
                 </geometry>
                 <material name="orange"/>
@@ -77,8 +77,8 @@
                 <geometry>
                     <xacro:if value="${mirror_dae == True}">
-                        <mesh filename="package://laikago_description/meshes/thigh.dae" scale="1 1 1"/>
+                        <mesh filename="package://arena-simulation-setup/robot/laikago/meshes/thigh.dae" scale="1 1 1"/>
                     </xacro:if>
                     <xacro:if value="${mirror_dae == False}">
-                        <mesh filename="package://laikago_description/meshes/thigh_mirror.dae" scale="1 1 1"/>
+                        <mesh filename="package://arena-simulation-setup/robot/laikago/meshes/thigh_mirror.dae" scale="1 1 1"/>
                     </xacro:if>
                 </geometry>
@@ -112,5 +112,5 @@
                 <origin rpy="0 0 0" xyz="0 0 0"/>
                 <geometry>
-                    <mesh filename="package://laikago_description/meshes/calf.dae" scale="1 1 1"/>
+                    <mesh filename="package://arena-simulation-setup/robot/laikago/meshes/calf.dae" scale="1 1 1"/>
                 </geometry>
                 <material name="orange"/>

Commit message: tweaks

File: robot/laikago/urdf/laikago.urdf.xacro (robot description, xacro)
@@ -2,8 +2,8 @@
 <robot name="laikago" xmlns:xacro="http://www.ros.org/wiki/xacro">
     <xacro:arg name="DEBUG" default="false"/>
-    <xacro:include filename="$(find arena-simulation-setup)/robot/laikago/xacro/const.xacro"/>
-    <xacro:include filename="$(find arena-simulation-setup)/robot/laikago/xacro/materials.xacro"/>
-    <xacro:include filename="$(find arena-simulation-setup)/robot/laikago/xacro/leg.xacro"/>
-    <xacro:include filename="$(find arena-simulation-setup)/robot/laikago/xacro/gazebo.xacro"/>
+    <xacro:include filename="$(find arena-simulation-setup)/robot/laikago/urdf/const.xacro"/>
+    <xacro:include filename="$(find arena-simulation-setup)/robot/laikago/urdf/materials.xacro"/>
+    <xacro:include filename="$(find arena-simulation-setup)/robot/laikago/urdf/leg.xacro"/>
+    <xacro:include filename="$(find arena-simulation-setup)/robot/laikago/urdf/gazebo.xacro"/>
     <!-- Rollover Protection mode will add an additional stick on the top, use "true" or "false" to switch it. -->
     <xacro:property name="rolloverProtection" value="false"/>
@@ -34,5 +34,5 @@
             <origin rpy="0 0 0" xyz="0 0 0"/>
             <geometry>
-                <mesh filename="package://arena-simulation-setup/robot/laikago/meshes/trunk.dae" scale="1 1 1"/>
+                <mesh filename="package://arena-simulation-setup/robot/laikago/urdf/meshes/trunk.dae" scale="1 1 1"/>
             </geometry>
             <material name="orange"/>

File: robot/laikago/urdf/leg.xacro (robot description, xacro)
@@ -1,5 +1,5 @@
 <?xml version="1.0"?>
 <robot xmlns:xacro="http://www.ros.org/wiki/xacro">
-    <xacro:include filename="$(find arena-simulation-setup)/robot/laikago/xacro/transmission.xacro"/>
+    <xacro:include filename="$(find arena-simulation-setup)/robot/laikago/urdf/transmission.xacro"/>
     <xacro:macro name="leg" params="name mirror mirror_dae front_hind front_hind_dae *origin">
         <joint name="${name}_hip_joint" type="revolute">
@@ -31,5 +31,5 @@
                 </xacro:if>
                 <geometry>
-                    <mesh filename="package://arena-simulation-setup/robot/laikago/meshes/hip.dae" scale="1 1 1"/>
+                    <mesh filename="package://arena-simulation-setup/robot/laikago/urdf/meshes/hip.dae" scale="1 1 1"/>
                 </geometry>
                 <material name="orange"/>
@@ -77,8 +77,8 @@
                 <geometry>
                     <xacro:if value="${mirror_dae == True}">
-                        <mesh filename="package://arena-simulation-setup/robot/laikago/meshes/thigh.dae" scale="1 1 1"/>
+                        <mesh filename="package://arena-simulation-setup/robot/laikago/urdf/meshes/thigh.dae" scale="1 1 1"/>
                     </xacro:if>
                     <xacro:if value="${mirror_dae == False}">
-                        <mesh filename="package://arena-simulation-setup/robot/laikago/meshes/thigh_mirror.dae" scale="1 1 1"/>
+                        <mesh filename="package://arena-simulation-setup/robot/laikago/urdf/meshes/thigh_mirror.dae" scale="1 1 1"/>
                     </xacro:if>
                 </geometry>
@@ -112,5 +112,5 @@
                 <origin rpy="0 0 0" xyz="0 0 0"/>
                 <geometry>
-                    <mesh filename="package://arena-simulation-setup/robot/laikago/meshes/calf.dae" scale="1 1 1"/>
+                    <mesh filename="package://arena-simulation-setup/robot/laikago/urdf/meshes/calf.dae" scale="1 1 1"/>
                 </geometry>
                 <material name="orange"/>
