Commit message: integrate laikago

File: robot/laikago/urdf/gazebo.xacro (robot description, xacro)
@@ -1,8 +1,9 @@
 <?xml version="1.0"?>
-<robot>
+<robot xmlns:xacro="http://www.ros.org/wiki/xacro">
+    <xacro:arg name="robot_namespace" default="laikago"/>
     <!-- ros_control plugin -->
     <gazebo>
         <plugin name="gazebo_ros_control" filename="libgazebo_ros_control.so">
-            <robotNamespace>/laikago_gazebo</robotNamespace>
+            <robotNamespace>$(arg robot_namespace)</robotNamespace>
             <robotSimType>gazebo_ros_control/DefaultRobotHWSim</robotSimType>
         </plugin>

File: robot/laikago/urdf/laikago.urdf.xacro (robot description, xacro)
@@ -6,4 +6,5 @@
     <xacro:include filename="$(find arena-simulation-setup)/robot/laikago/urdf/leg.xacro"/>
     <xacro:include filename="$(find arena-simulation-setup)/robot/laikago/urdf/gazebo.xacro"/>
+    <xacro:include filename="$(find arena-simulation-setup)/robot/laikago/urdf/lidar.xacro"/>
     <!-- Rollover Protection mode will add an additional stick on the top, use "true" or "false" to switch it. -->
     <xacro:property name="rolloverProtection" value="false"/>
@@ -119,3 +120,6 @@
         <origin rpy="0 0 0" xyz="${-leg_offset_x} ${leg_offset_y} 0"/>
     </xacro:leg>
+    <xacro:lidar parent="trunk">
+        <origin rpy="0 0 0" xyz="0.05 0 0.125"/>
+    </xacro:lidar>
 </robot>
